File: powerdist/battprot_v0.1.kicad_sch (KiCad schematic)
At the start: 0 parts

Commit message: lab 30/09
Parts:
- added U4: BQ7791508PWR, TSSOP24_4P4X7P8_THT_TEX, symbol BQ7791508:BQ7791508PWR
Changed lines of the file:
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@@
 	(generator_version "8.0")
 	(paper "A4")
+	(symbol
+		(lib_id "BQ7791508:BQ7791508PWR")
+		(at 128.27 52.07 0)
+		(unit 1)
+		(exclude_from_sim no)
+		(in_bom yes)
+		(on_board yes)
+		(dnp no)
+		(fields_autoplaced yes)
+		(property "Reference" "U4"
+			(at 148.59 41.91 0)
+			(effects
+				(font
+					(size 1.524 1.524)
+				)
+			)
+		)
+		(property "Value" "BQ7791508PWR"
+			(at 148.59 44.45 0)
+			(effects
+				(font
+					(size 1.524 1.524)
+				)
+			)
+		)
+		(property "Footprint" "TSSOP24_4P4X7P8_THT_TEX"
+			(at 128.27 52.07 0)
+			(effects
+				(font
+					(size 1.27 1.27)
+					(italic yes)
+				)
+				(hide yes)
+			)
+		)
+		(property "Datasheet" "https://www.ti.com/lit/gpn/bq77915"
+			(at 128.27 52.07 0)
+			(effects
+				(font
+					(size 1.27 1.27)
+					(italic yes)
+				)
+				(hide yes)
+			)
+		)
+		(property "Description" ""
+			(at 128.27 52.07 0)
+			(effects
+				(font
+					(size 1.27 1.27)
+				)
+				(hide yes)
+			)
+		)
+		(pin "18"
+		)
+		(pin "5"
+		)
+		(pin "1"
+		)
+		(pin "11"
+		)
+		(pin "8"
+		)
+		(pin "22"
+		)
+		(pin "4"
+		)
+		(pin "21"
+		)
+		(pin "2"
+		)
+		(pin "24"
+		)
+		(pin "6"
+		)
+		(pin "10"
+		)
+		(pin "20"
+		)
+		(pin "9"
+		)
+		(pin "15"
+		)
+		(pin "19"
+		)
+		(pin "3"
+		)
+		(pin "16"
+		)
+		(pin "23"
+		)
+		(pin "12"
+		)
+		(pin "13"
+		)
+		(pin "7"
+		)
+		(pin "17"
+		)
+		(pin "14"
+		)
+		(instances
+			(project ""
+				(path "/d8b3361c-0c6a-4299-baf2-0b5966ddedfb/754cc4f7-7309-49ec-a85a-88e49e6da610/1b151f5e-d113-49d8-a928-351d73068788"
+					(reference "U4")
+					(unit 1)
+				)
+			)
+		)
+	)
 )
