File: powerdist/battprot_v0.1.kicad_sch (KiCad schematic)
At the start: 31 parts, among them Q3 NMOS, Q4 NMOS, SW3 SW_DPDT_x2, U2 BQ7791508PWR

Commit message: local 12/10
Connections:
- net 1BATT- renamed CELLGND
- net 1BATT1 renamed CELL1
- net 1BATT2 renamed CELL2
- net 1BATT3 renamed CELL3
- net 1BATT4 renamed CELL4
- net 1VC0 renamed VC0
- net 1VC1 renamed VC1
- net 1VC2 renamed VC2
- net 1VC3 renamed VC3
- net 1VC4 renamed VC4
- net AVDD1 renamed AVDD
- net CCFG1 renamed CCFG
- net CHG1 renamed CHG
- net DSG1 renamed DSG
- net PSRN1 renamed PSRN
- net PSRP1 renamed PSRP
- net TS1 renamed TS
- net VDD1 renamed VDD
- net Vbatt1 renamed Vbatt
- net Vtb1 renamed Vtb
Other:
- note added: "!DS12.1!"
- note added: "!DS12.2!"
- note added: "!DS12.5!"
- note added: "CTRC/CTRD outputs"
- note added: "turn to high side"
- note removed: "xBATT- is GND: GNDPWR may float when FETs disabled"
- moved on the sheet: C14, C15, C16, D6, D7, Q3, Q4, R21, R22, R27, R28, R29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
