File: powerdist/battcharge_v0.1.kicad_sch (KiCad schematic)
At the start: 45 parts, among them Q1 SI7617DN, Q2 SI7617DN, Q3 SIS412DN, Q4 SIS412DN, Q5 SI7617DN, U1 BQ24610

Commit message: local 30/09
Parts:
- added R58: 76.8k, symbol Device:R_Small_US
- added R59: 26.1k, symbol Device:R_Small_US
- added R64: 90.9k, symbol Device:R_Small_US
- added R65: 13k, symbol Device:R_Small_US
- added SW1: SW_DPDT_x2, symbol Switch:SW_DPDT_x2
- R10: value 57.6k -> 120k
- R11: value 44.2k -> 33k
- R12: value 120k -> 57.6k
- R13: value 33k -> 44.2k
- renumbered C2 to C29, C3 to C30, C10 to C31, C4 to C32, C13 to C33, C14 to C34, C9 to C35, C6 to C36, C7 to C37, C8 to C38, C1 to C39, C11 to C40, C5 to C41, C12 to C42, D3 to D10, D4 to D11, D1 to D12, D2 to D9, L1 to L3, Q1 to Q11, Q2 to Q12, Q3 to Q13, Q4 to Q14, Q5 to Q15, R8 to R39, R15 to R40, R16 to R41, R9 to R42, R4 to R43, R3 to R44, R17 to R45, R18 to R46, R19 to R47, R14 to R52, R2 to R53, R1 to R54, R7 to R55, R6 to R56, R5 to R57, TH1 to TH3, U1 to U3
Connections:
- net GND: now also R59.2, R65.2
- net Vref1: now also SW1.2 (B), SW1.5 (B); no longer R10.1, R12.1
- net 1ISET2: now reaches R10.2, R11.1
- net 1ISET2: now also U3.15 (ISET2), R64.2, R65.1; no longer U3.11 (ISET1)
- net 1ISET1: now reaches R12.2, R13.1
- net 1ISET1: now also U3.11 (ISET1), R58.2, R59.1; no longer U3.15 (ISET2)
- new net: R12.1, SW1.3 (C)
- new net: R58.1, SW1.1 (A)
- new net: R10.1, SW1.6 (C)
- new net: R64.1, SW1.4 (A)
Other:
- note added: "!CELL DEPENDENT!"
- note added: "!DEPENDENT ON ESR!"
- note added: "ACTIVE?"
- note added: "CHG?"
- note added: "D=63% L=3.3uH IHLP2525CZ (high Isat) dI=2.4A Ichg=4.2A C=40u (datasheet)"
- note added: "DONE?"
- note added: "Ichg=4.2A Viset1=0.84V R8=0.84/3.3=25.4% R8=26.1k,R7=76.8k"
- note added: "Ipcg=Iterm=0.42A Viset2=0.42V R6=0.42/3.3=12.7% R6=13k,R5=90.9k"
- note added: "R2/R1=7or5 R1=100k"
- note added: "Vin=20V 3S 4.2Ah Vbatt=12.6V=4*4.2V Pchg=46.62W"
- note added: "hell to RC: Cin ftw high ESR high C"
- note added: "high ESR?"
- note removed: "!ESR>1M!"
- note removed: "R2/R1=7 R1=100k"
- note removed: "hell to RC: Cin ftw"
- moved on the sheet: C29, C30, C31, C36, C37, C38, C40, C41, D10, D11, D12, D9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

Commit message: lab 30/09
Parts:
- added R70: 500k, symbol Device:R_Small_US
- added SW1: SW_SPDT, symbol Switch:SW_SPDT
- renumbered C29 to C1, C38 to C10, C39 to C11, C40 to C12, C41 to C13, C42 to C14, C30 to C2, C31 to C3, C32 to C4, C33 to C5, C34 to C6, C35 to C7, C36 to C8, C37 to C9, D9 to D1, D10 to D2, D11 to D3, D12 to D4, L3 to L1, Q11 to Q1, Q12 to Q2, Q13 to Q3, Q14 to Q4, Q15 to Q5, R39 to R1, R52 to R14, R53 to R15, R54 to R16, R55 to R17, R56 to R18, R57 to R19, R40 to R2, R41 to R3, R42 to R4, R43 to R5, R44 to R6, R45 to R7, R46 to R8, R47 to R9, SW1 to SW2, TH3 to TH1, U3 to U1
Connections:
- net Vbatt1: now also SW1.2 (B); no longer R15.1
- net Vfb: now also R70.2
- new net: R15.1, SW1.1 (A)
- new net: R70.1, SW1.3 (C)
Other:
- note added: "!HIGH ESR!"
- note added: "!SAME AS SW1!"
- note added: "!SAME AS SW2!"
- note removed: "!CELL DEPENDENT!"
- note removed: "!DEPENDENT ON ESR!"
- moved on the sheet: C10, C11, C12, C13, C14, D4, L1, Q3, Q4, Q5, R10, R11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

Commit message: lab 02/10
Parts:
- renumbered C1 to C15, C2 to C16, C4 to C17, C3 to C18, C5 to C19, C6 to C20, C7 to C21, C8 to C22, C9 to C23, C10 to C24, C11 to C25, C12 to C26, C13 to C27, C14 to C28, D1 to D5, D2 to D6, D3 to D7, D4 to D8, L1 to L2, Q5 to Q10, Q1 to Q6, Q2 to Q7, Q3 to Q8, Q4 to Q9, R1 to R20, R2 to R21, R3 to R22, R4 to R23, R5 to R24, R6 to R25, R7 to R26, R8 to R27, R9 to R28, R14 to R29, R15 to R30, R16 to R31, R12 to R32, R13 to R33, R58 to R34, R59 to R35, R17 to R36, R10 to R37, R11 to R38, R18 to R39, R19 to R40, R64 to R41, R65 to R42, R70 to R71, SW1 to SW4, TH1 to TH2, U1 to U2
