File: powerdist/battprotSLAV_v0.1.kicad_sch (KiCad schematic)
At the start: 1 part, among them U4 BQ7791508PWR

Commit message: lab 02/10
Parts:
- removed U4: BQ7791508PWR, TSSOP24_4P4X7P8_THT_TEX, symbol BQ7791508:BQ7791508PWR
- added C45: C_Small, symbol Device:C_Small
- added U6: BQ7791508PWR, TSSOP24_4P4X7P8_THT_TEX, symbol BQ7791508:BQ7791508PWR
Changed lines of the file:
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@@
 	(generator_version "8.0")
 	(paper "A4")
+	(global_label "Vbatt1"
+		(shape input)
+		(at 119.38 60.96 180)
+		(fields_autoplaced yes)
+		(effects
+			(font
+				(size 1.27 1.27)
+			)
+			(justify right)
+		)
+		(property "Intersheetrefs" "${INTERSHEET_REFS}"
+			(at 110.3473 60.96 0)
+			(effects
+				(font
+					(size 1.27 1.27)
+				)
+				(justify right)
+				(hide yes)
+			)
+		)
+	)
+	(symbol
+		(lib_id "Device:C_Small")
+		(at 123.19 66.04 0)
+		(unit 1)
+		(exclude_from_sim no)
+		(in_bom yes)
+		(on_board yes)
+		(dnp no)
+		(property "Reference" "C45"
+			(at 120.65 64.7762 0)
+			(effects
+				(font
+					(size 1.27 1.27)
+				)
+				(justify right)
+			)
+		)
+		(property "Value" "C_Small"
+			(at 120.65 67.3162 0)
+			(effects
+				(font
+					(size 1.27 1.27)
+				)
+				(justify right)
+			)
+		)
+		(property "Footprint" ""
+			(at 123.19 66.04 0)
+			(effects
+				(font
+					(size 1.27 1.27)
+				)
+				(hide yes)
+			)
+		)
+		(property "Datasheet" "~"
+			(at 123.19 66.04 0)
+			(effects
+				(font
+					(size 1.27 1.27)
+				)
+				(hide yes)
+			)
+		)
+		(property "Description" "Unpolarized capacitor, small symbol"
+			(at 123.19 66.04 0)
+			(effects
+				(font
+					(size 1.27 1.27)
+				)
+				(hide yes)
+			)
+		)
+		(pin "1"
+		)
+		(pin "2"
+		)
+		(instances
+			(project "powerdist"
+				(path "/d8b3361c-0c6a-4299-baf2-0b5966ddedfb/754cc4f7-7309-49ec-a85a-88e49e6da610/03bbebe4-b14f-4c2c-8c4b-910fc22197eb"
+					(reference "C45")
+					(unit 1)
+				)
+				(path "/d8b3361c-0c6a-4299-baf2-0b5966ddedfb/754cc4f7-7309-49ec-a85a-88e49e6da610/db06460c-6b9d-4c4a-9584-c744e6276cab"
+					(reference "C44")
+					(unit 1)
+				)
+			)
+		)
+	)
 	(symbol
 		(lib_id "BQ7791508:BQ7791508PWR")
-		(at 128.27 52.07 0)
+		(at 133.35 60.96 0)
 		(unit 1)
 		(exclude_from_sim no)
@@
 		(dnp no)
 		(fields_autoplaced yes)
-		(property "Reference" "U4"
-			(at 148.59 41.91 0)
+		(property "Reference" "U6"
+			(at 153.67 50.8 0)
 			(effects
 				(font
@@
 		)
 		(property "Value" "BQ7791508PWR"
-			(at 148.59 44.45 0)
+			(at 153.67 53.34 0)
 			(effects
 				(font
@@
 		)
 		(property "Footprint" "TSSOP24_4P4X7P8_THT_TEX"
-			(at 128.27 52.07 0)
+			(at 154.432 96.266 0)
 			(effects
 				(font
@@
 		)
 		(property "Datasheet" "https://www.ti.com/lit/gpn/bq77915"
-			(at 128.27 52.07 0)
+			(at 153.924 98.552 0)
 			(effects
 				(font
@@
 		)
 		(property "Description" ""
-			(at 128.27 52.07 0)
-			(effects
-				(font
-					(size 1.27 1.27)
-				)
-				(hide yes)
-			)
+			(at 133.35 60.96 0)
+			(effects
+				(font
+					(size 1.27 1.27)
+				)
+				(hide yes)
+			)
+		)
+		(pin "13"
+		)
+		(pin "15"
+		)
+		(pin "7"
+		)
+		(pin "6"
+		)
+		(pin "21"
+		)
+		(pin "19"
+		)
+		(pin "14"
+		)
+		(pin "9"
+		)
+		(pin "12"
+		)
+		(pin "2"
+		)
+		(pin "20"
+		)
+		(pin "22"
+		)
+		(pin "1"
+		)
+		(pin "10"
+		)
+		(pin "24"
+		)
+		(pin "4"
+		)
+		(pin "11"
+		)
+		(pin "8"
+		)
+		(pin "5"
+		)
+		(pin "16"
 		)
 		(pin "18"
 		)
-		(pin "5"
-		)
-		(pin "1"
-		)
-		(pin "11"
-		)
-		(pin "8"
-		)
-		(pin "22"
-		)
-		(pin "4"
-		)
-		(pin "21"
-		)
-		(pin "2"
-		)
-		(pin "24"
-		)
-		(pin "6"
-		)
-		(pin "10"
-		)
-		(pin "20"
-		)
-		(pin "9"
-		)
-		(pin "15"
-		)
-		(pin "19"
+		(pin "17"
+		)
+		(pin "23"
 		)
 		(pin "3"
 		)
-		(pin "16"
-		)
-		(pin "23"
-		)
-		(pin "12"
-		)
-		(pin "13"
-		)
-		(pin "7"
-		)
-		(pin "17"
-		)
-		(pin "14"
-		)
 		(instances
-			(project ""
-				(path "/d8b3361c-0c6a-4299-baf2-0b5966ddedfb/754cc4f7-7309-49ec-a85a-88e49e6da610/1b151f5e-d113-49d8-a928-351d73068788"
-					(reference "U4")
-					(unit 1)
-				)
+			(project "powerdist"
+				(path "/d8b3361c-0c6a-4299-baf2-0b5966ddedfb/754cc4f7-7309-49ec-a85a-88e49e6da610/03bbebe4-b14f-4c2c-8c4b-910fc22197eb"
+					(reference "U6")
+					(unit 1)
+				)
+				(path "/d8b3361c-0c6a-4299-baf2-0b5966ddedfb/754cc4f7-7309-49ec-a85a-88e49e6da610/db06460c-6b9d-4c4a-9584-c744e6276cab"
+					(reference "U5")
+					(unit 1)
+				)
