File: powerdist/battprotSLAV_v0.1.kicad_sch (KiCad schematic)
At the start: 2 parts, among them U6 BQ7791508PWR

Commit message: lab 09/10
Parts:
- renumbered C51 to C59, U6 to U7
Changed lines of the file:
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@@
 		(on_board yes)
 		(dnp no)
-		(property "Reference" "C51"
+		(property "Reference" "C59"
 			(at 120.65 64.7762 0)
 			(effects
@@
 			(project "powerdist"
 				(path "/d8b3361c-0c6a-4299-baf2-0b5966ddedfb/754cc4f7-7309-49ec-a85a-88e49e6da610/03bbebe4-b14f-4c2c-8c4b-910fc22197eb"
-					(reference "C51")
+					(reference "C59")
 					(unit 1)
 				)
 				(path "/d8b3361c-0c6a-4299-baf2-0b5966ddedfb/754cc4f7-7309-49ec-a85a-88e49e6da610/db06460c-6b9d-4c4a-9584-c744e6276cab"
-					(reference "C50")
+					(reference "C58")
 					(unit 1)
 				)
@@
 		(dnp no)
 		(fields_autoplaced yes)
-		(property "Reference" "U6"
+		(property "Reference" "U7"
 			(at 153.67 50.8 0)
 			(effects
@@
 			(project "powerdist"
 				(path "/d8b3361c-0c6a-4299-baf2-0b5966ddedfb/754cc4f7-7309-49ec-a85a-88e49e6da610/03bbebe4-b14f-4c2c-8c4b-910fc22197eb"
+					(reference "U7")
+					(unit 1)
+				)
+				(path "/d8b3361c-0c6a-4299-baf2-0b5966ddedfb/754cc4f7-7309-49ec-a85a-88e49e6da610/db06460c-6b9d-4c4a-9584-c744e6276cab"
 					(reference "U6")
 					(unit 1)
 				)
-				(path "/d8b3361c-0c6a-4299-baf2-0b5966ddedfb/754cc4f7-7309-49ec-a85a-88e49e6da610/db06460c-6b9d-4c4a-9584-c744e6276cab"
-					(reference "U5")
-					(unit 1)
-				)
