File: powerdist/battprotMSTR_v0.1.kicad_sch (KiCad schematic)
At the start: 2 parts, among them U4 BQ7791508PWR

Commit message: local 07/10
Parts:
- removed C43: C_Small, symbol Device:C_Small
- removed U4: BQ7791508PWR, TSSOP24_4P4X7P8_THT_TEX, symbol BQ7791508:BQ7791508PWR
- added C15, C16, C17, C18, C19, C52, C53, C54: 100n, symbol Device:C_Small
- added C20, C21: C_Small, symbol Device:C_Small
- added D13: D_Zener_Small_Filled, symbol Device:D_Zener_Small_Filled
- added D14: ~, symbol Device:D_Small_Filled
- added Q16, Q17: NMOS, symbol Simulation_SPICE:NMOS
- added R25, R26, R27, R28, R30: 36, symbol Device:R_Small_US
- added R29, R31: R_Small_US, symbol Device:R_Small_US
- added R80: 4m, symbol Device:R_Small_US
- added R81, R82: 100, symbol Device:R_Small_US
- added R83, R84, R86: 1M, symbol Device:R_Small_US
- added R85: 4.5k, symbol Device:R_Small_US
- added R87: 750k, symbol Device:R_Small_US
- added SW3, SW8: SW_DPDT_x2, symbol Switch:SW_DPDT_x2
- added U2: BQ7791508PWR, TSSOP24_4P4X7P8_THT_TEX, symbol BQ7791508:BQ7791508PWR
Connections:
- net Vbatt1: now also R29.1
- new net: Q17.3 (S), R80.1, R82.2, R83.1
- new net: Q16.1 (D), Q17.1 (D)
- new net: Q17.2 (G), R83.2, R85.1
- new net: C15.1, R25.2, SW3.3 (C)
- new net: D13.1 (K), D14.1 (K), Q16.2 (G), R84.1, R86.2
- new net: R87.2, U2.17 (OCDP)
- new net: R31.2, U2.22 (PRES)
- new net 1BATT-: C18.2, C19.1, C20.2, C21.2, C53.1, C54.2, R30.1, R87.1, SW8.4 (A), U2.16 (CBI), U2.23 (CTRC), U2.24 (CTRD), U2.9 (VSS)
- new net 1BATT1: R28.1
- new net 1BATT2: R27.1
- new net 1BATT3: R26.1
- new net 1BATT4: R25.1
- new net 1VC0: C19.2, R30.2, U2.8 (VC0)
- new net 1VC1: C17.2, C18.1, R28.2, U2.7 (VC1)
- new net 1VC2: C16.2, C17.1, R27.2, U2.6 (VC2)
- new net 1VC3: C15.2, C16.1, R26.2, SW3.1 (A), U2.5 (VC3)
- new net 1VC4: SW3.2 (B), U2.3 (VC5), U2.4 (VC4)
- new net AVDD1: C21.1, SW8.6 (C), U2.2 (AVDD)
- new net CCFG1: SW8.5 (B), U2.20 (CCFG)
- new net CHG1: D14.2 (A), R86.1, U2.13 (CHG)
- new net DSG1: R85.2, U2.12 (DSG)
- new net GNDPWR: D13.2 (A), Q16.3 (S), R84.2
- new net PSRN1: C52.1, C54.1, R82.1, U2.11 (SRN)
- new net PSRP1: C52.2, C53.2, R81.2, U2.10 (SRP)
- new net VDD1: C20.1, R29.2, R31.1, U2.1 (VDD)
- new net Vbatt1-: R80.2, R81.1
- no-connect marks 0 -> 2
Other:
- note added: "!LOW Req!"
- note added: "Ibal=50mA<<Iterm=0.72A or 0.42A Vcell=4.2V Rbal=12 Vcell/Ibal=2*Rin+Rbal Rin=.5(Vcell/Ibal-Rbal) Rin=36"
- note added: "LD?"
- note added: "Vocd1=70mV let Iocd1=14A (138W@9.9V, 229W@16.4V) Rsns=5m Vocd2=140mV Iocd2=28A Vscd=300mV Iscd=60A Vocc=60mV Iocc=12A"
- note added: "charg or prot TS?"
- note added: "xBATT- is GND: GNDPWR may float when FETs disabled"
- title: (none) -> Battery Protection Circuit: Master Mode

Commit message: lab 09/10
Parts:
- D7: renamed from D13; value D_Zener_Small_Filled -> ~
- renumbered C53 to C14, C52 to C15, C54 to C16, C15 to C17, C17 to C18, C16 to C20, C18 to C21, C20 to C22, C21 to C23, D14 to D6, Q17 to Q3, Q16 to Q4, R81 to R21, R80 to R22, R25 to R23, R26 to R24, R27 to R25, R28 to R26, R30 to R27, R82 to R28, R83 to R29, R85 to R30, R86 to R31, R84 to R32, R29 to R33, R31 to R34, R87 to R35, SW8 to SW3
Connections:
- net 1BATT-: now also U2.14 (LD)
- net VDD1: now also R34.2; no longer R34.1
- net Vbatt1-: now also R22.1, R28.2; no longer R21.1, R22.2
- net at Q3.3 (S), R29.1: now also R21.1, R22.2; no longer R22.1, R28.2
- net at U2.22 (PRES): now also R34.1; no longer R34.2
- net TS1: now reaches U2.18 (TS)
- net Vtb1: now reaches U2.19 (VTB)
Other:
- note added: "LD never disconnected"
- note removed: "LD?"
- note removed: "charg or prot TS?"
- moved on the sheet: C14, C15, C16, C17, C18, C19, C20, C21, D6, D7, Q3, Q4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
