File: powerdist/v0.1.kicad_sch (KiCad schematic)
At the start: 0 parts

Commit message: local 30/09
Parts:
- added BATT1, BATT2, BATT3, INPUT1: Conn_01x02_Socket, symbol Connector:Conn_01x02_Socket
- added BATT1S1, BATT2S1, BATT3S1: Conn_01x04_Pin, symbol Connector:Conn_01x04_Pin
- added BATT1S2, BATT2S2, BATT3S2: Conn_01x03_Pin, symbol Connector:Conn_01x03_Pin
- added F1: Fuse_Small, symbol Device:Fuse_Small
Connections:
- new net Vbatt1: F1.2
Other:
- sheet battcharger3S_v0.1_1 renamed battcharger3S_1
- sheet battcharger3S_v0.1_2 renamed battcharger3S_2
- sheet battcharger4S_v0.1 renamed battcharger4S
- sheet battprot_v0.1 renamed battprot
- sheet buck5V1_v0.1 renamed buck5V1
- sheet buck7V5_v0.1 renamed buck7V5
- sheet buckboost_v0.1 renamed buckboost
- sheet battcharger3S_1: file battcharge3S_v0.1.kicad_sch -> battcharge_v0.1.kicad_sch
- sheet battcharger3S_2: file battcharge3S_v0.1.kicad_sch -> battcharge_v0.1.kicad_sch
- sheet battcharger4S: file battcharge4S_v0.1.kicad_sch -> battcharge_v0.1.kicad_sch
- sheet battprot: file battprot.kicad_sch -> battprot_v0.1.kicad_sch
- sheet buck5V1: file buck5V1.kicad_sch -> buck5V1_v0.1.kicad_sch
- sheet buck7V5: file buck7V5.kicad_sch -> buck7V5_v0.1.kicad_sch
- sheet buckboost: file buckboost.kicad_sch -> buckboost_v0.1.kicad_sch
- note added: "TODO: battery connector (POLARITY!) + fuse holder"
- note removed: "TODO: battery connector + fuse holder"
- title: (none) -> v0.1

Commit message: lab 30/09
Other:
- removed sheet battcharger3S_1
- removed sheet battcharger3S_2
- added sheet battcharger3S1 (battcharge_v0.1.kicad_sch)
- added sheet battcharger3S2 (battcharge_v0.1.kicad_sch)
Changed lines of the file:
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@@
+	)
+	(sheet
+		(at 13.97 53.34)
+		(size 59.69 33.02)
+		(fields_autoplaced yes)
+		(stroke
+			(width 0.1524)
+			(type solid)
+		)
+		(fill
+			(color 0 0 0 0.0000)
+		)
+		(property "Sheetname" "battcharger3S1"
+			(at 13.97 52.6284 0)
+			(effects
+				(font
+					(size 1.27 1.27)
+				)
+				(justify left bottom)
+			)
+		)
+		(property "Sheetfile" "battcharge_v0.1.kicad_sch"
+			(at 13.97 86.9446 0)
+			(effects
+				(font
+					(size 1.27 1.27)
+				)
+				(justify left top)
+			)
+		)
+		(instances
+			(project "powerdist"
+				(path "/d8b3361c-0c6a-4299-baf2-0b5966ddedfb/754cc4f7-7309-49ec-a85a-88e49e6da610"
+					(page "8")
+				)
+			)
+		)
 	)
 	(sheet
@@
 			(color 0 0 0 0.0000)
 		)
-		(property "Sheetname" "battcharger3S_2"
+		(property "Sheetname" "battcharger3S2"
 			(at 13.97 90.7284 0)
 			(effects
@@
 			)
 		)
+		(property "Field2" ""
+			(at 13.97 91.44 0)
+			(effects
+				(font
+					(size 1.27 1.27)
+				)
+				(hide yes)
+			)
+		)
 		(instances
 			(project "powerdist"
 				(path "/d8b3361c-0c6a-4299-baf2-0b5966ddedfb/754cc4f7-7309-49ec-a85a-88e49e6da610"
-					(page "8")
+					(page "9")
 				)
 			)
@@
 				)
 			)
-		)
-	)
-	(sheet
-		(at 13.97 53.34)
-		(size 59.69 33.02)
-		(fields_autoplaced yes)
-		(stroke
-			(width 0.1524)
-			(type solid)
-		)
-		(fill
-			(color 0 0 0 0.0000)
-		)
-		(property "Sheetname" "battcharger3S_1"
-			(at 13.97 52.6284 0)
-			(effects
-				(font
-					(size 1.27 1.27)
-				)
-				(justify left bottom)
-			)
-		)
-		(property "Sheetfile" "battcharge_v0.1.kicad_sch"
-			(at 13.97 86.9446 0)
-			(effects
-				(font
-					(size 1.27 1.27)
-				)
-				(justify left top)
-			)
-		)
-		(instances
-			(project "powerdist"
-				(path "/d8b3361c-0c6a-4299-baf2-0b5966ddedfb/754cc4f7-7309-49ec-a85a-88e49e6da610"
-					(page "3")
-				)
-			)

Commit message: lab 02/10
Parts:
- added F2, F3: Fuse_Small, symbol Device:Fuse_Small
- BATT1S1, BATT2S1, BATT3S1: symbol Connector:Conn_01x04_Pin -> Connector:Conn_01x05_Pin
- BATT1S2, BATT2S2, BATT3S2: symbol Connector:Conn_01x03_Pin -> Connector:Conn_01x04_Pin
Connections:
- net GNDPWR: now also BATT1.1 (Pin_1), BATT1S1.5 (Pin_5), BATT1S2.4 (Pin_4), BATT2.1 (Pin_1), BATT2S1.5 (Pin_5), BATT2S2.4 (Pin_4), BATT3.1 (Pin_1), BATT3S1.5 (Pin_5), BATT3S2.4 (Pin_4), INPUT1.1 (Pin_1)
- net VAA: now also INPUT1.2 (Pin_2)
- net Vbatt2: now also F2.2
- net Vbatt3: now also F3.2
- net at BATT1.2 (Pin_2): now also F1.1
- net at BATT2.2 (Pin_2): now also F2.1
- net 3BATT3: now reaches BATT3S2.1 (Pin_1)
- net 3BATT3: now also BATT3S1.2 (Pin_2)
- net 3BATT2: now reaches BATT3S2.2 (Pin_2)
- net 3BATT2: now also BATT3S1.3 (Pin_3)
- net 3BATT1: now reaches BATT3S2.3 (Pin_3)
- net 3BATT1: now also BATT3S1.4 (Pin_4)
- net 3BATT4: now reaches BATT3S1.1 (Pin_1)
- net 2BATT4: now reaches BATT2S1.1 (Pin_1)
- net 2BATT3: now reaches BATT2S1.2 (Pin_2)
- net 2BATT3: now also BATT2S2.1 (Pin_1)
- net 2BATT2: now reaches BATT2S1.3 (Pin_3)
- net 2BATT2: now also BATT2S2.2 (Pin_2)
- net 2BATT1: now reaches BATT2S1.4 (Pin_4)
- net 2BATT1: now also BATT2S2.3 (Pin_3)
- net at BATT3.2 (Pin_2): now also F3.1
- net 1BATT3: now reaches BATT1S2.1 (Pin_1)
- net 1BATT3: now also BATT1S1.2 (Pin_2)
- net 1BATT2: now reaches BATT1S2.2 (Pin_2)
- net 1BATT2: now also BATT1S1.3 (Pin_3)
- net 1BATT1: now reaches BATT1S2.3 (Pin_3)
- net 1BATT1: now also BATT1S1.4 (Pin_4)
- net 1BATT4: now reaches BATT1S1.1 (Pin_1)
Other:
- sheet battprot renamed battprot1
- added sheet battprot2 (battprotSLAV_v0.1.kicad_sch)
- added sheet battprot3 (battprotSLAV_v0.1.kicad_sch)
- sheet battprot1: file battprot_v0.1.kicad_sch -> battprotMSTR_v0.1.kicad_sch
- note added: "!11A CAPABLE!"
- moved on the sheet: BATT1, BATT2, BATT3, F1, INPUT1

Commit message: local 07/10
Connections:
- net GNDPWR: no longer BATT1.1 (Pin_1), BATT1S1.5 (Pin_5), BATT1S2.4 (Pin_4), BATT2.1 (Pin_1), BATT2S1.5 (Pin_5), BATT2S2.4 (Pin_4), BATT3.1 (Pin_1), BATT3S1.5 (Pin_5), BATT3S2.4 (Pin_4)
- new net 1BATT-: BATT1S1.5 (Pin_5), BATT1S2.4 (Pin_4)
- new net 2BATT-: BATT2S1.5 (Pin_5), BATT2S2.4 (Pin_4)
- new net 3BATT-: BATT3S1.5 (Pin_5), BATT3S2.4 (Pin_4)
- new net Vbatt1-: BATT1.1 (Pin_1)
- new net Vbatt2-: BATT2.1 (Pin_1)
- new net Vbatt3-: BATT3.1 (Pin_1)
Other:
- moved on the sheet: INPUT1

Commit message: lab 09/10
Parts:
- added CHGSTAT: Conn_01x02_Pin, symbol Connector:Conn_01x02_Pin
- added R6: 10k, symbol Device:R_Small_US
- added TH1: 103AT-11, symbol Device:Thermistor_US
Connections:
- net 1BATT-: now also TH1.1
- net 1STAT2: now also CHGSTAT.2 (Pin_2)
- new net 1STAT1: CHGSTAT.1 (Pin_1)
- new net TS1: R6.2, TH1.2
- new net Vtb1: R6.1
Other:
- sheet battcharger3S1: file battcharge_v0.1.kicad_sch -> battcharge_v0.2.kicad_sch
- sheet battcharger3S2: file battcharge_v0.1.kicad_sch -> battcharge_v0.2.kicad_sch
- sheet battcharger4S: file battcharge_v0.1.kicad_sch -> battcharge_v0.2.kicad_sch
- note added: "all open-drain to RPI? or ~EN buck-boost?"

Commit message: local 12/10
Parts:
- added D19: 1N4148, symbol Device:D_Small_Filled
- added R119, R44: 10k, symbol Device:R_Small_US
- renumbered CHGSTAT to CHGSTAT1, R6 to R21
Connections:
- net 1BATT-: no longer TH1.1
- net VAA: now also R119.1, R44.1
- net 1STAT1: no longer names the net of CHGSTAT1.1 (Pin_1)
- net 1STAT2: no longer names the net of CHGSTAT1.2 (Pin_2)
- net TS1: no longer names the net of R21.2, TH1.2
- net Vtb1: no longer names the net of R21.1
- new net CE: D19.1 (K), R44.2
- new net CHG: D19.2 (A), R119.2
Other:
- sheet battcharger3S1 ports: added CE, STAT1, STAT2, Vout; removed none
- sheet battcharger3S2 ports: added CE, STAT1, STAT2, Vout; removed none
- sheet battcharger4S ports: added CE, STAT1, STAT2, Vout; removed none
- sheet battprot1: file battprotMSTR_v0.1.kicad_sch -> battprot_v0.2.kicad_sch
- sheet battprot1 ports: added CELL1, CELL2, CELL3, CELL4, CELLGND, CHG, TS, Vbatt, Vbatt-, Vin, Vtb; removed none
- sheet battprot2: file battprotSLAV_v0.1.kicad_sch -> battprot_v0.2.kicad_sch
- sheet battprot2 ports: added CELL1, CELL2, CELL3, CELL4, CELLGND, CHG, TS, Vbatt, Vbatt-, Vin, Vtb; removed none
- sheet battprot3: file battprotSLAV_v0.1.kicad_sch -> battprot_v0.2.kicad_sch
- sheet battprot3 ports: added CELL1, CELL2, CELL3, CELL4, CELLGND, CHG, TS, Vbatt, Vbatt-, Vin, Vtb; removed none
- sheet buck5V1: file buck5V1_v0.1.kicad_sch -> buck_v0.1.kicad_sch
- sheet buck7V5: file buck7V5_v0.1.kicad_sch -> buck_v0.1.kicad_sch
- sheet buckboost ports: added EN; removed none
- note removed: "!11A CAPABLE!"
- moved on the sheet: R21, TH1
