File: powerdist/v0.1.kicad_sch (KiCad schematic)
At the start: 29 parts

Commit message: local 14/10
Parts:
- renumbered BATT1S2 to BATT3S1, BATT2S2 to BATT3S2, BATT3S2 to BATT3S3, BATT1S1 to BATT4S1, BATT2S1 to BATT4S2, BATT3S1 to BATT4S3, INPUT1 to J1, 12Vout1 to J2, 7V5out1 to J3, 5V1out1 to J4
Changed lines of the file:
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@@
 		(dnp no)
 		(fields_autoplaced yes)
-		(property "Reference" "5V1out1"
+		(property "Reference" "J4"
 			(at 152.4 189.2299 0)
 			(effects
@@
 			(project "powerdist"
 				(path "/d8b3361c-0c6a-4299-baf2-0b5966ddedfb/754cc4f7-7309-49ec-a85a-88e49e6da610"
-					(reference "5V1out1")
+					(reference "J4")
 					(unit 1)
 				)
@@
 		(dnp no)
 		(fields_autoplaced yes)
-		(property "Reference" "#FLG01"
+		(property "Reference" "#FLG03"
 			(at 218.44 161.925 0)
 			(effects
@@
 			(project "powerdist"
 				(path "/d8b3361c-0c6a-4299-baf2-0b5966ddedfb/754cc4f7-7309-49ec-a85a-88e49e6da610"
-					(reference "#FLG01")
+					(reference "#FLG03")
 					(unit 1)
 				)
@@
 		(dnp no)
 		(fields_autoplaced yes)
-		(property "Reference" "12Vout1"
+		(property "Reference" "J2"
 			(at 152.4 161.2899 0)
 			(effects
@@
 			(project "powerdist"
 				(path "/d8b3361c-0c6a-4299-baf2-0b5966ddedfb/754cc4f7-7309-49ec-a85a-88e49e6da610"
-					(reference "12Vout1")
+					(reference "J2")
 					(unit 1)
 				)
@@
 		(dnp no)
 		(fields_autoplaced yes)
-		(property "Reference" "7V5out1"
+		(property "Reference" "J3"
 			(at 152.4 175.2599 0)
 			(effects
@@
 			(project "powerdist"
 				(path "/d8b3361c-0c6a-4299-baf2-0b5966ddedfb/754cc4f7-7309-49ec-a85a-88e49e6da610"
-					(reference "7V5out1")
+					(reference "J3")
 					(unit 1)
 				)
@@
 		(dnp no)
 		(fields_autoplaced yes)
-		(property "Reference" "#FLG03"
+		(property "Reference" "#FLG05"
 			(at 238.76 161.925 0)
 			(effects
@@
 			(project "powerdist"
 				(path "/d8b3361c-0c6a-4299-baf2-0b5966ddedfb/754cc4f7-7309-49ec-a85a-88e49e6da610"
-					(reference "#FLG03")
+					(reference "#FLG05")
 					(unit 1)
 				)
@@
 		(dnp no)
 		(fields_autoplaced yes)
-		(property "Reference" "BATT3S2"
+		(property "Reference" "BATT3S3"
 			(at 106.045 182.88 0)
 			(effects
@@
 			(project "powerdist"
 				(path "/d8b3361c-0c6a-4299-baf2-0b5966ddedfb/754cc4f7-7309-49ec-a85a-88e49e6da610"
-					(reference "BATT3S2")
+					(reference "BATT3S3")
 					(unit 1)
 				)
@@
 		(dnp no)
 		(fields_autoplaced yes)
-		(property "Reference" "BATT3S1"
+		(property "Reference" "BATT4S3"
 			(at 106.045 166.37 0)
 			(effects
@@
 			(project "powerdist"
 				(path "/d8b3361c-0c6a-4299-baf2-0b5966ddedfb/754cc4f7-7309-49ec-a85a-88e49e6da610"
-					(reference "BATT3S1")
+					(reference "BATT4S3")
 					(unit 1)
 				)
@@
 		(dnp no)
 		(fields_autoplaced yes)
-		(property "Reference" "BATT2S1"
+		(property "Reference" "BATT4S2"
 			(at 65.405 166.37 0)
 			(effects
@@
 			(project "powerdist"
 				(path "/d8b3361c-0c6a-4299-baf2-0b5966ddedfb/754cc4f7-7309-49ec-a85a-88e49e6da610"
-					(reference "BATT2S1")
+					(reference "BATT4S2")
 					(unit 1)
 				)
@@
 		(dnp no)
 		(fields_autoplaced yes)
-		(property "Reference" "#FLG04"
+		(property "Reference" "#FLG06"
 			(at 248.92 161.925 0)
 			(effects
@@
 			(project "powerdist"
 				(path "/d8b3361c-0c6a-4299-baf2-0b5966ddedfb/754cc4f7-7309-49ec-a85a-88e49e6da610"
-					(reference "#FLG04")
+					(reference "#FLG06")
 					(unit 1)
 				)
@@
 		(dnp no)
 		(fields_autoplaced yes)
-		(property "Reference" "#FLG05"
+		(property "Reference" "#FLG07"
 			(at 259.08 161.925 0)
 			(effects
@@
 			(project "powerdist"
 				(path "/d8b3361c-0c6a-4299-baf2-0b5966ddedfb/754cc4f7-7309-49ec-a85a-88e49e6da610"
-					(reference "#FLG05")
+					(reference "#FLG07")
 					(unit 1)
 				)
@@
 		(dnp no)
 		(fields_autoplaced yes)
-		(property "Reference" "BATT1S2"
+		(property "Reference" "BATT3S1"
 			(at 24.765 182.88 0)
 			(effects
@@
 			(project ""
 				(path "/d8b3361c-0c6a-4299-baf2-0b5966ddedfb/754cc4f7-7309-49ec-a85a-88e49e6da610"
-					(reference "BATT1S2")
+					(reference "BATT3S1")
 					(unit 1)
 				)
@@
 		(dnp no)
 		(fields_autoplaced yes)
-		(property "Reference" "INPUT1"
+		(property "Reference" "J1"
 			(at 27.305 138.43 0)
 			(effects
@@
 			(project ""
 				(path "/d8b3361c-0c6a-4299-baf2-0b5966ddedfb/754cc4f7-7309-49ec-a85a-88e49e6da610"
-					(reference "INPUT1")
+					(reference "J1")
 					(unit 1)
 				)
@@
 		(dnp no)
 		(fields_autoplaced yes)
-		(property "Reference" "BATT2S2"
+		(property "Reference" "BATT3S2"
 			(at 65.405 182.88 0)
 			(effects
@@
 			(project "powerdist"
 				(path "/d8b3361c-0c6a-4299-baf2-0b5966ddedfb/754cc4f7-7309-49ec-a85a-88e49e6da610"
-					(reference "BATT2S2")
+					(reference "BATT3S2")
 					(unit 1)
 				)
@@
 		(dnp no)
 		(fields_autoplaced yes)
-		(property "Reference" "BATT1S1"
+		(property "Reference" "BATT4S1"
 			(at 24.765 166.37 0)
 			(effects
@@
 			(project ""
 				(path "/d8b3361c-0c6a-4299-baf2-0b5966ddedfb/754cc4f7-7309-49ec-a85a-88e49e6da610"
-					(reference "BATT1S1")
+					(reference "BATT4S1")
 					(unit 1)
 				)
@@
 		(dnp no)
 		(fields_autoplaced yes)
-		(property "Reference" "#FLG02"
+		(property "Reference" "#FLG04"
 			(at 228.6 161.925 0)
 			(effects
@@
 			(project "powerdist"
 				(path "/d8b3361c-0c6a-4299-baf2-0b5966ddedfb/754cc4f7-7309-49ec-a85a-88e49e6da610"
-					(reference "#FLG02")
+					(reference "#FLG04")
 					(unit 1)
 				)
@@
 		(dnp no)
 		(fields_autoplaced yes)
-		(property "Reference" "#FLG07"
+		(property "Reference" "#FLG08"
 			(at 279.4 158.115 0)
 			(effects
@@
 			(project "powerdist"
 				(path "/d8b3361c-0c6a-4299-baf2-0b5966ddedfb/754cc4f7-7309-49ec-a85a-88e49e6da610"
-					(reference "#FLG07")
+					(reference "#FLG08")
 					(unit 1)
 				)

Commit message: local 19/10
Parts:
- added Q23, Q24, Q25: SIS412DN, symbol Simulation_SPICE:NMOS
- added R127, R128, R129: 100k, symbol Device:R_Small_US
- BATT1, BATT2, BATT3: footprint (none) -> Connector:Banana_Jack_2Pin
- BATT3S1, BATT3S2, BATT3S3: footprint (none) -> Connector_JST:JST_XH_B4B-XH-AM_1x04_P2.50mm_Vertical
- BATT4S1, BATT4S2, BATT4S3: footprint (none) -> Connector_JST:JST_XH_B5B-XH-AM_1x05_P2.50mm_Vertical
- J1, J2, J3, J4: symbol Connector:Conn_01x02_Socket -> Connector:Screw_Terminal_01x02
- R24: value 20k -> 75k
- renumbered C12 to C16, C13 to C17, C14 to C18
Connections:
- net Vbatt1: now also Q23.2 (G), R127.1
- net Vbatt1-: now also Q23.3 (S), R127.2; no longer BATT1.1 (Pin_1)
- net Vbatt2: now also Q24.2 (G), R128.1
- net Vbatt2-: now also Q24.3 (S), R128.2; no longer BATT2.1 (Pin_1)
- net Vbatt3: now also Q25.2 (G), R129.1
- net Vbatt3-: now also Q25.3 (S), R129.2; no longer BATT3.1 (Pin_1)
- new net: BATT1.1 (Pin_1), Q23.1 (D)
- new net: BATT2.1 (Pin_1), Q24.1 (D)
- new net: BATT3.1 (Pin_1), Q25.1 (D)
Other:
- moved on the sheet: BATT1, BATT2, BATT3, BATT3S1, BATT3S2, BATT3S3, BATT4S1, BATT4S2, BATT4S3, C16, C17, C18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

Commit message: lab 20/10
Parts:
- removed F1, F2, F3: Fuse_Small, symbol Device:Fuse_Small
- removed Q24, Q25: SIS412DN, symbol Simulation_SPICE:NMOS
- removed R127, R128, R129: 100k, symbol Device:R_Small_US
- added D6, D8, D9: BZT52, symbol Device:D_Zener_Small_Filled
- added F1, F2, F3: 3544-2, powerdist:CONN_3544-2_KEY, symbol 3544-2:3544-2
- added Q4, Q5: SI4178DY, symbol Simulation_SPICE:NMOS
- added R22, R23, R25: 1k, symbol Device:R_Small_US
- Q3: renamed from Q23; value SIS412DN -> SI4178DY
- renumbered D5 to D4, D6 to D5, R22 to R24, R23 to R26, R24 to R27
Connections:
- net Vbatt1: now also F1.3, F1.4, R22.1; no longer Q3.2 (G)
- net Vbatt1-: now also D6.2 (A)
- net Vbatt2: now also F2.3, F2.4, R23.1
- net Vbatt2-: now also D8.2 (A), Q4.3 (S)
- net Vbatt3: now also F3.3, F3.4, R25.1
- net Vbatt3-: now also D9.2 (A), Q5.3 (S)
- net at BATT1.2 (Pin_2): now also F1.1, F1.2
- net at BATT3.2 (Pin_2): now also F3.1, F3.2
- net at BATT2.1 (Pin_1): now also Q4.1 (D)
- net at BATT2.2 (Pin_2): now also F2.1, F2.2
- net at BATT3.1 (Pin_1): now also Q5.1 (D)
- new net: D8.1 (K), Q4.2 (G), R23.2
- new net: D9.1 (K), Q5.2 (G), R25.2
- new net: D6.1 (K), Q3.2 (G), R22.2
Other:
- moved on the sheet: BATT1, BATT2, BATT3, BATT3S1, BATT3S2, BATT3S3, BATT4S1, BATT4S2, BATT4S3, C16, C17, C18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

Commit message: lab 21/10
Parts:
- D10: renamed from D9; footprint (none) -> Diode_SMD:D_SOD-123
- D5: renamed from D4; footprint (none) -> Diode_SMD:D_SOD-123
- D6: renamed from D5; footprint (none) -> Diode_SMD:D_SOD-123
- D7: renamed from D6; footprint (none) -> Diode_SMD:D_SOD-123
- D8: renamed from D7; footprint (none) -> Diode_SMD:D_SOD-123
- D9: renamed from D8; footprint (none) -> Diode_SMD:D_SOD-123
- J1, J2, J3, J4: footprint (none) -> TerminalBlock:TerminalBlock_bornier-2_P5.08mm
- L2, L3: footprint (none) -> Inductor_SMD:L_Vishay_IHLP-5050
- R20, R21, R22, R23, R24, R25, R26, R27: footprint (none) -> Resistor_SMD:R_0603_1608Metric
Other:
- note added: "ALL INDUCTORS IHLP5050FDxxxRxMA1"
Changed lines of the file:
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@@
 		)
 	)
+	(text "ALL INDUCTORS IHLP5050FDxxxRxMA1"
+		(exclude_from_sim no)
+		(at 256.794 178.562 0)
+		(effects
+			(font
+				(size 1.27 1.27)
+			)
+		)
+	)
 	(label "CE2"
 		(at 22.86 111.76 180)
@@
 			)
 		)
-		(property "Footprint" ""
+		(property "Footprint" "TerminalBlock:TerminalBlock_bornier-2_P5.08mm"
 			(at 251.46 48.26 0)
 			(effects
@@
 			)
 		)
-		(property "Footprint" ""
+		(property "Footprint" "Resistor_SMD:R_0603_1608Metric"
 			(at 105.41 24.13 0)
 			(effects
@@
 			)
 		)
-		(property "Footprint" ""
+		(property "Footprint" "Resistor_SMD:R_0603_1608Metric"
 			(at 22.86 152.4 0)
 			(effects
@@
 		(on_board yes)
 		(dnp no)
-		(property "Reference" "D5"
+		(property "Reference" "D6"
 			(at 19.05 162.56 0)
 			(effects
@@
 			)
 		)
-		(property "Footprint" ""
+		(property "Footprint" "Diode_SMD:D_SOD-123"
 			(at 19.05 156.21 90)
 			(effects
@@
 			(project "powerdist"
 				(path "/d8b3361c-0c6a-4299-baf2-0b5966ddedfb/754cc4f7-7309-49ec-a85a-88e49e6da610"
-					(reference "D5")
+					(reference "D6")
 					(unit 1)
 				)
@@
 			)
 		)
-		(property "Footprint" ""
+		(property "Footprint" "TerminalBlock:TerminalBlock_bornier-2_P5.08mm"
 			(at 251.46 20.32 0)
 			(effects
@@
 			)
 		)
-		(property "Footprint" ""
+		(property "Footprint" "TerminalBlock:TerminalBlock_bornier-2_P5.08mm"
 			(at 251.46 34.29 0)
 			(effects
@@
 			)
 		)
-		(property "Footprint" ""
+		(property "Footprint" "Resistor_SMD:R_0603_1608Metric"
 			(at 256.54 149.86 0)
 			(effects
@@
 			)
 		)
-		(property "Footprint" ""
+		(property "Footprint" "Resistor_SMD:R_0603_1608Metric"
 			(at 166.37 24.13 0)
 			(effects
@@
 		(on_board yes)
 		(dnp no)
-		(property "Reference" "D7"
+		(property "Reference" "D8"
 			(at 71.12 81.28 0)
 			(effects
@@
 			)
 		)
-		(property "Footprint" ""
+		(property "Footprint" "Diode_SMD:D_SOD-123"
 			(at 71.12 87.63 90)
 			(effects
@@
 			(project "powerdist"
 				(path "/d8b3361c-0c6a-4299-baf2-0b5966ddedfb/754cc4f7-7309-49ec-a85a-88e49e6da610"
-					(reference "D7")
+					(reference "D8")
 					(unit 1)
 				)
@@
 			)
 		)
-		(property "Footprint" ""
+		(property "Footprint" "Resistor_SMD:R_0603_1608Metric"
 			(at 256.54 111.76 0)
 			(effects
@@
 			)
 		)
-		(property "Footprint" ""
+		(property "Footprint" "Inductor_SMD:L_Vishay_IHLP-5050"
 			(at 256.54 127 0)
 			(effects
@@
 			)
 		)
-		(property "Footprint" ""
+		(property "Footprint" "TerminalBlock:TerminalBlock_bornier-2_P5.08mm"
 			(at 208.28 25.4 0)
 			(effects
@@
 			)
 		)
-		(property "Footprint" ""
+		(property "Footprint" "Resistor_SMD:R_0603_1608Metric"
 			(at 152.4 114.3 0)
 			(effects
@@
 			)
 		)
-		(property "Footprint" ""
+		(property "Footprint" "Resistor_SMD:R_0603_1608Metric"
 			(at 44.45 24.13 0)
 			(effects
@@
 		(on_board yes)
 		(dnp no)
-		(property "Reference" "D4"
+		(property "Reference" "D5"
 			(at 19.05 124.46 0)
 			(effects
@@
 			)
 		)
-		(property "Footprint" ""
+		(property "Footprint" "Diode_SMD:D_SOD-123"
 			(at 19.05 118.11 90)
 			(effects
@@
 			(project "powerdist"
 				(path "/d8b3361c-0c6a-4299-baf2-0b5966ddedfb/754cc4f7-7309-49ec-a85a-88e49e6da610"
-					(reference "D4")
+					(reference "D5")
 					(unit 1)
 				)
@@
 		(dnp no)
 		(fields_autoplaced yes)
-		(property "Reference" "D9"
+		(property "Reference" "D10"
 			(at 173.99 29.2099 90)
 			(effects
@@
 			)
 		)
-		(property "Footprint" ""
+		(property "Footprint" "Diode_SMD:D_SOD-123"
 			(at 171.45 30.48 90)
 			(effects
@@
 			(project "powerdist"
 				(path "/d8b3361c-0c6a-4299-baf2-0b5966ddedfb/754cc4f7-7309-49ec-a85a-88e49e6da610"
-					(reference "D9")
+					(reference "D10")
 					(unit 1)
 				)
@@
 		(dnp no)
 		(fields_autoplaced yes)
-		(property "Reference" "D6"
+		(property "Reference" "D7"
 			(at 52.07 29.2099 90)
 			(effects
@@
 			)
 		)
-		(property "Footprint" ""
+		(property "Footprint" "Diode_SMD:D_SOD-123"
 			(at 49.53 30.48 90)
 			(effects
@@
 			(project ""
 				(path "/d8b3361c-0c6a-4299-baf2-0b5966ddedfb/754cc4f7-7309-49ec-a85a-88e49e6da610"
-					(reference "D6")
+					(reference "D7")
 					(unit 1)
 				)
@@
 		(dnp no)
 		(fields_autoplaced yes)
-		(property "Reference" "D8"
+		(property "Reference" "D9"
 			(at 113.03 29.2099 90)
 			(effects
@@
 			)
 		)
-		(property "Footprint" ""
+		(property "Footprint" "Diode_SMD:D_SOD-123"
 			(at 110.49 30.48 90)
 			(effects
@@
 			(project "powerdist"
 				(path "/d8b3361c-0c6a-4299-baf2-0b5966ddedfb/754cc4f7-7309-49ec-a85a-88e49e6da610"
-					(reference "D8")
+					(reference "D9")
 					(unit 1)
 				)
@@
 			)
 		)
-		(property "Footprint" ""
+		(property "Footprint" "Resistor_SMD:R_0603_1608Metric"
 			(at 22.86 114.3 0)
 			(effects
@@
 			)
 		)
-		(property "Footprint" ""
+		(property "Footprint" "Inductor_SMD:L_Vishay_IHLP-5050"
 			(at 256.54 88.9 0)
 			(effects

Commit message: lab 23/10
Parts:
- C16, C17, C18: footprint (none) -> Capacitor_SMD:C_1206_3216Metric; symbol Device:C_Polarized_Small_US -> Device:C_Small
- Q3, Q4, Q5: footprint (none) -> Package_SO:PowerPAK_SO-8_Single; symbol Simulation_SPICE:NMOS -> Transistor_FET:Si7336ADP
- renumbered D8 to D10, D7 to D5, D9 to D6, D10 to D7, D5 to D8, D6 to D9, R22 to R20, R23 to R21, R25 to R22, R20 to R23, R21 to R24, R24 to R25
Connections:
- net Vbatt1-: now also Q3.1 (S), Q3.2 (S)
- net Vbatt2-: now also Q4.1 (S), Q4.2 (S)
- net Vbatt3-: now also Q5.1 (S), Q5.2 (S)
- net at BATT1.1 (Pin_1): now also Q3.5 (D); no longer Q3.1 (D)
- net at D6.1 (K), R21.2: now also Q4.4 (G); no longer Q4.2 (G)
- net at BATT3.1 (Pin_1): now also Q5.5 (D); no longer Q5.1 (D)
- net at D7.1 (K), R22.2: now also Q5.4 (G); no longer Q5.2 (G)
- net at BATT2.1 (Pin_1): now also Q4.5 (D); no longer Q4.1 (D)
- net at D5.1 (K), R20.2: now also Q3.4 (G); no longer Q3.2 (G)
Other:
- moved on the sheet: BATT1, BATT2, BATT3, BATT3S1, BATT3S2, BATT3S3, BATT4S1, BATT4S2, BATT4S3, D10, D5, D6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
