File: powerdist/battcharge_v0.2.kicad_sch (KiCad schematic)
At the start: 42 parts, among them Q1 SIS412DN, Q2 SIS412DN, SW1 SW_SPDT, SW2 SW_DPDT_x2, U1 BQ24610

Commit message: local 12/10
Parts:
- removed C2: 100u, symbol Device:C_Polarized_Small_US
- removed D4: ~, symbol Device:D_Schottky_Small_Filled
- removed R2: 1, symbol Device:R_Small_US
- added R55: 100k, symbol Device:R_Small_US
- C44: renamed from C1; value 100u -> 2.2u
- R50: renamed from R1; value 1 -> 2
- renumbered C3 to C46, C4 to C47, C5 to C48, C7 to C49, C8 to C50, C9 to C51, C10 to C52, C11 to C53, C12 to C54, C13 to C55, D2 to D10, D3 to D11, D5 to D13, D1 to D9, L1 to L3, Q1 to Q11, Q2 to Q12, R3 to R52, R4 to R53, R5 to R54, R7 to R56, R46 to R57, R9 to R58, R10 to R59, R11 to R60, R12 to R61, R13 to R62, R14 to R63, R15 to R64, R16 to R65, R17 to R66, R18 to R67, R19 to R68, R20 to R69, SW1 to SW4, SW2 to SW5, U1 to U4
Connections:
- net Vchg1 is gone; now on net VAA: C46.1, C53.1, Q11.1 (D), U4.1 (ACN), U4.2 (ACP), U4.24 (VCC)
- net GND: now also R55.2
- net VAA: now also R55.1
- net 1ISET1 renamed ISET1
- net 1ISET2 renamed ISET2
- net 1STAT1 renamed STAT1
- net 1STAT2 renamed STAT2
- net BTST1 renamed BTST
- net BTST: now also C54.1; no longer C54.2
- net CHG1 renamed CE
- net CSRP1 renamed CSRP
- net HIDRV1 renamed HIDRV
- net LODRV1 renamed LODRV
- net PG1 renamed PG
- net PH1 renamed PH
- net PH: now also C54.2; no longer C54.1
- net REGN1 renamed REGN
- net Vbatt1 renamed Vout
- net Vout: no longer C52.1, SW4.2 (B)
- net Vref1 renamed Vref
- net ~BATDRV1: no longer names the net of U4.23 (~{BATDRV})
- new net Vbatt: C52.1, SW4.2 (B)
- no-connect marks 1 -> 2
Other:
- note added: "0.42A"
- note added: "0.72A"
- note added: "3S"
- note added: "4.2A"
- note added: "4S"
- note added: "7.2A"
- note added: "use battprot's TS->CHG->CE"
- note removed: "use battprot's TS->CHG"
- moved on the sheet: C44, C46, C47, C48, C49, C50, C51, C54, D13, R50, R56, R57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

Commit message: local 13/10
Parts:
- renumbered C44 to C56, C46 to C57, C47 to C58, C48 to C59, C49 to C60, C50 to C61, C51 to C62, C52 to C63, C53 to C64, C54 to C65, C55 to C66, D9 to D12, D10 to D13, D11 to D14, D13 to D15, L3 to L5, R50 to R57, R52 to R58, R53 to R59, R54 to R60, R55 to R61, R56 to R62, R57 to R63, R58 to R64, R59 to R65, R60 to R66, R61 to R67, R62 to R68, R63 to R69, R64 to R70, R65 to R71, R66 to R72, R67 to R73, R68 to R74, R69 to R75, U4 to U6
Connections:
- net Vbatt is gone; now on net Vout: C63.1, SW4.2 (B)
Other:
- note removed: "!HIGH ESR!"
- note removed: "!SAME AS SW1!"
- note removed: "!SAME AS SW2!"

Commit message: local 19/10
Parts:
- added C69, C72, C73, C74: 10u, Capacitor_SMD:C_1206_3216Metric, symbol Device:C_Small
- C60: renamed from C56; footprint (none) -> Capacitor_SMD:C_1206_3216Metric; symbol Device:C_Polarized_Small_US -> Device:C_Small
- C61: renamed from C57; footprint (none) -> Capacitor_SMD:C_0603_1608Metric
- C62: renamed from C58; footprint (none) -> Capacitor_SMD:C_0603_1608Metric
- C63: renamed from C59; footprint (none) -> Capacitor_SMD:C_0603_1608Metric
- C64: renamed from C60; footprint (none) -> Capacitor_SMD:C_0603_1608Metric
- C65: renamed from C61; footprint (none) -> Capacitor_SMD:C_0603_1608Metric
- C66: renamed from C62; footprint (none) -> Capacitor_SMD:C_0603_1608Metric
- C67: renamed from C63; footprint (none) -> Capacitor_SMD:C_0603_1608Metric
- C68: renamed from C64; value 20u -> 10u; footprint (none) -> Capacitor_SMD:C_1206_3216Metric; symbol Device:C_Polarized_Small_US -> Device:C_Small
- C70: renamed from C65; footprint (none) -> Capacitor_SMD:C_0603_1608Metric
- C71: renamed from C66; value 40u -> 10u; footprint (none) -> Capacitor_SMD:C_1206_3216Metric; symbol Device:C_Polarized_Small_US -> Device:C_Small
- renumbered R73 to R71, R71 to R72, R72 to R73
Connections:
- net GND: now also C69.2, C72.2, C73.2, C74.2
- net VAA: now also C69.1
- net Vout: now also C72.1, C73.1, C74.1
Other:
- note removed: "!DS12.3!"
- moved on the sheet: C61, C62, C63, C64, C65, C66, C67, C70, D15, L5, Q11, Q12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

Commit message: lab 20/10
Parts:
- added D4B1: BAT54C, symbol Device:D_Schottky_Small_Filled
- D17: renamed from D15; value ~ -> BAT54C
- renumbered C68 to C67, C69 to C68, C67 to C69, D12 to D14, D13 to D15, D14 to D16, Q11 to Q14, Q12 to Q15, R57 to R60, R58 to R61, R59 to R62, R60 to R63, R61 to R64, R62 to R65, R63 to R66, R64 to R67, R65 to R68, R66 to R69, R67 to R70, R68 to R71, R69 to R72, R70 to R73, R71 to R74, R72 to R75, R73 to R76, R74 to R77, R75 to R78
Connections:
- net BTST: now also D4B1.1 (K)
- net REGN: now also D4B1.2 (A)
Other:
- moved on the sheet: C61, C62, C63, C64, C65, C66, C67, C68, C70, D17, R65, R66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

Commit message: lab 21/10
Parts:
- removed D17, D4B1: BAT54C, symbol Device:D_Schottky_Small_Filled
- added D4: BAT54CL, Package_TO_SOT_SMD:SOT-23-3, symbol D_Schottky_AAK_Parallel_Small_Filled:D_Schottky_Dual_CommonCathode_AAK_Parallel
- D15: renamed from D14; footprint (none) -> LED_SMD:LED_0603_1608Metric
- D16: renamed from D15; footprint (none) -> LED_SMD:LED_0603_1608Metric
- D17: renamed from D16; footprint (none) -> LED_SMD:LED_0603_1608Metric
- L5: footprint (none) -> Inductor_SMD:L_Vishay_IHLP-5050
- R60, R61, R62, R63, R64, R65, R66, R67, R68, R69, R70, R71, R72, R73, R74, R75, R76, R77, R78: footprint (none) -> Resistor_SMD:R_0603_1608Metric
- SW4: value SW_SPDT -> OS102011M; footprint (none) -> Button_Switch_THT:SW_Slide_SPDT_Straight_CK_OS102011MS2Q
- SW5: value SW_DPDT_x2 -> JS202011CQN; footprint (none) -> Button_Switch_THT:SW_CK_JS202011CQN_DPDT_Straight
Connections:
- net BTST: now also D4.3 (K)
- net REGN: now also D4.1 (A), D4.2 (A)
Other:
- note added: "D=63% L=3.3uH dI=2.4A Ichg=4.2A C=40u (datasheet)"
- note added: "D=84% L=3.3uH dI=1.4A Ichg=7.2A C=40u (datasheet)"
- note removed: "D=63% L=3.3uH IHLP2525CZ (high Isat) dI=2.4A Ichg=4.2A C=40u (datasheet)"
- note removed: "D=84% L=3.3uH IHLP2525CZ (high Isat) dI=1.4A Ichg=7.2A C=40u (datasheet)"
- moved on the sheet: C70

Commit message: lab 23/10
Parts:
- Q14, Q15: footprint (none) -> Package_SO:Vishay_PowerPAK_1212-8_Single; symbol Simulation_SPICE:NMOS -> Transistor_FET:SiS454DN
- renumbered D4 to D18
Connections:
- net GND: now also Q15.1 (S), Q15.2 (S)
- net HIDRV: now also Q14.4 (G); no longer Q14.2 (G)
- net LODRV: now also Q15.4 (G); no longer Q15.2 (G)
- net PH: now also Q14.1 (S), Q14.2 (S), Q15.5 (D); no longer Q15.1 (D)
- net VAA: now also Q14.5 (D); no longer Q14.1 (D)
Changed lines of the file:
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@@
 	)
 	(symbol
-		(lib_id "Simulation_SPICE:NMOS")
+		(lib_id "Transistor_FET:SiS454DN")
 		(at 238.76 43.18 0)
 		(unit 1)
@@
 			)
 		)
-		(property "Footprint" ""
-			(at 243.84 40.64 0)
+		(property "Footprint" "Package_SO:Vishay_PowerPAK_1212-8_Single"
+			(at 243.84 45.085 0)
 			(effects
 				(font
 					(size 1.27 1.27)
+					(italic yes)
 				)
+				(justify left)
 				(hide yes)
 			)
 		)
-		(property "Datasheet" "https://ngspice.sourceforge.io/docs/ngspice-html-manual/manual.xhtml#cha_MOSFETs"
-			(at 238.76 55.88 0)
+		(property "Datasheet" "https://www.vishay.com/docs/66707/sis454dn.pdf"
+			(at 243.84 46.99 0)
 			(effects
 				(font
 					(size 1.27 1.27)
 				)
+				(justify left)
 				(hide yes)
 			)
 		)
-		(property "Description" "N-MOSFET transistor, drain/source/gate"
+		(property "Description" "35A Id, 20V Vds, N-Channel MOSFET, PowerPAK 1212-8 Single"
 			(at 238.76 43.18 0)
 			(effects
@@
 		(pin "1"
 		)
+		(pin "5"
+		)
+		(pin "4"
+		)
 		(instances
 			(project "powerdist"
@@
 	)
 	(symbol
-		(lib_id "Simulation_SPICE:NMOS")
+		(lib_id "Transistor_FET:SiS454DN")
 		(at 238.76 24.13 0)
 		(unit 1)
@@
 			)
 		)
-		(property "Footprint" ""
-			(at 243.84 21.59 0)
+		(property "Footprint" "Package_SO:Vishay_PowerPAK_1212-8_Single"
+			(at 243.84 26.035 0)
 			(effects
 				(font
 					(size 1.27 1.27)
+					(italic yes)
 				)
+				(justify left)
 				(hide yes)
 			)
 		)
-		(property "Datasheet" "https://ngspice.sourceforge.io/docs/ngspice-html-manual/manual.xhtml#cha_MOSFETs"
-			(at 238.76 36.83 0)
+		(property "Datasheet" "https://www.vishay.com/docs/66707/sis454dn.pdf"
+			(at 243.84 27.94 0)
 			(effects
 				(font
 					(size 1.27 1.27)
 				)
+				(justify left)
 				(hide yes)
 			)
 		)
-		(property "Description" "N-MOSFET transistor, drain/source/gate"
+		(property "Description" "35A Id, 20V Vds, N-Channel MOSFET, PowerPAK 1212-8 Single"
 			(at 238.76 24.13 0)
 			(effects
@@
 		(pin "1"
 		)
+		(pin "4"
+		)
+		(pin "5"
+		)
 		(instances
 			(project "powerdist"
@@
 		(dnp no)
 		(fields_autoplaced yes)
-		(property "Reference" "D4"
+		(property "Reference" "D18"
 			(at 229.87 28.0037 90)
 			(effects

Commit message: local 26/10
Parts:
- renumbered C66 to C10, C67 to C11, C68 to C12, C69 to C13, C70 to C14, C71 to C15, C72 to C16, C73 to C17, C74 to C18, C60 to C4, C61 to C5, C62 to C6, C63 to C7, C64 to C8, C65 to C9, D15 to D12, D16 to D13, D17 to D14, D18 to D15, L5 to L3, Q15 to Q10, Q14 to Q9, R60 to R12, R61 to R13, R62 to R14, R63 to R15, R64 to R16, R65 to R17, R66 to R18, R67 to R19, R68 to R20, R69 to R21, R70 to R22, R71 to R23, R72 to R24, R73 to R25, R74 to R26, R75 to R27, R76 to R28, R77 to R29, R78 to R30, SW4 to SW1, SW5 to SW2, U6 to U1
Connections:
- net VAA: no longer C11.1, C12.1, C5.1, Q9.5 (D), R12.1, U1.1 (ACN), U1.2 (ACP), U1.24 (VCC)
- new net Vin: C11.1, C12.1, C5.1, Q9.5 (D), R12.1, U1.1 (ACN), U1.2 (ACP), U1.24 (VCC)
