File: powerdist/battcharge_v0.2.kicad_sch (KiCad schematic)
At the start: 44 parts, among them Q10 SIS412DN, Q9 SIS412DN, SW1 OS102011M, SW2 JS202011CQN, U1 BQ24610

Commit message: lab 27/10
Parts:
- R26: footprint Resistor_SMD:R_0603_1608Metric -> Resistor_SMD:R_1206_3216Metric
Changed lines of the file:
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@@
 		(on_board yes)
 		(dnp no)
-		(fields_autoplaced yes)
 		(property "Reference" "L3"
 			(at 247.65 29.21 90)
@@
 			)
 		)
-		(property "Footprint" "Resistor_SMD:R_0603_1608Metric"
+		(property "Footprint" "Resistor_SMD:R_1206_3216Metric"
 			(at 256.54 34.29 0)
 			(effects

Commit message: lab 28/10
Parts:
- removed R16: 100k, Resistor_SMD:R_0603_1608Metric, symbol Device:R_Small_US
- R19: value 500k -> 700k
- R20: value 700k -> 500k
- R22: value 57.6k -> 76.8k
- R23: value 44.2k -> 26.1k
- R24: value 76.8k -> 57.6k
- R25: value 26.1k -> 44.2k
Connections:
- net CSRP: now also C10.1
- net Vout: no longer C10.1
Other:
- moved on the sheet: C10
Changed lines of the file:
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@@
 		)
 	)
-	(text "4.2A\n"
+	(text "7.2A"
 		(exclude_from_sim no)
 		(at 246.634 86.36 0)
@@
 		)
 	)
-	(text "3S"
+	(text "4S"
 		(exclude_from_sim no)
 		(at 200.66 81.026 0)
@@
 		)
 	)
-	(text "7.2A\n"
+	(text "4.2A\n"
 		(exclude_from_sim no)
 		(at 225.806 86.36 0)
@@
 	(text "!DS12.4!"
 		(exclude_from_sim no)
-		(at 138.43 58.674 0)
+		(at 138.43 57.658 0)
 		(effects
 			(font
@@
 	(text "!DS12.4!"
 		(exclude_from_sim no)
-		(at 138.43 65.532 0)
+		(at 128.778 62.992 0)
 		(effects
 			(font
@@
 		)
 	)
-	(text "4S"
+	(text "3S\n"
 		(exclude_from_sim no)
 		(at 190.5 81.026 0)
@@
 		(exclude_from_sim no)
 		(at 12.7 43.18 0)
-		(size 29.21 39.37)
+		(size 29.21 29.21)
 		(margins 0.9525 0.9525 0.9525 0.9525)
 		(stroke
@@
 	)
 	(junction
-		(at 39.37 69.85)
-		(diameter 0)
-		(color 0 0 0 0)
-	)
-	(junction
 		(at 264.16 34.29)
 		(diameter 0)
@@
 	)
 	(junction
+		(at 124.46 55.88)
+		(diameter 0)
+		(color 0 0 0 0)
+	)
+	(junction
 		(at 125.73 44.45)
 		(diameter 0)
@@
 	)
 	(junction
-		(at 127 62.23)
-		(diameter 0)
-		(color 0 0 0 0)
-	)
-	(junction
 		(at 259.08 41.91)
 		(diameter 0)
@@
 	(wire
 		(pts
-			(xy 127 63.5) (xy 127 62.23)
-		)
-		(stroke
-			(width 0)
-			(type default)
-		)
-	)
-	(wire
-		(pts
 			(xy 252.73 33.02) (xy 252.73 34.29)
 		)
@@
 	(wire
 		(pts
-			(xy 116.84 55.88) (xy 127 55.88)
+			(xy 116.84 55.88) (xy 124.46 55.88)
 		)
 		(stroke
@@
 	(wire
 		(pts
-			(xy 39.37 71.12) (xy 39.37 69.85)
-		)
-		(stroke
-			(width 0)
-			(type default)
-		)
-	)
-	(wire
-		(pts
-			(xy 127 62.23) (xy 134.62 62.23)
+			(xy 127 60.96) (xy 134.62 60.96)
 		)
 		(stroke
@@
 	(wire
 		(pts
+			(xy 124.46 55.88) (xy 127 55.88)
+		)
+		(stroke
+			(width 0)
+			(type default)
+		)
+	)
+	(wire
+		(pts
 			(xy 39.37 69.85) (xy 38.1 69.85)
 		)
@@
 	(wire
 		(pts
-			(xy 127 62.23) (xy 127 60.96)
-		)
-		(stroke
-			(width 0)
-			(type default)
-		)
-	)
-	(wire
-		(pts
 			(xy 208.28 19.05) (xy 241.3 19.05)
 		)
@@
 	(wire
 		(pts
+			(xy 124.46 55.88) (xy 124.46 63.5)
+		)
+		(stroke
+			(width 0)
+			(type default)
+		)
+	)
+	(wire
+		(pts
 			(xy 115.57 72.39) (xy 114.3 72.39)
 		)
@@
 	)
 	(label "CSRN"
-		(at 134.62 62.23 0)
+		(at 134.62 60.96 0)
 		(effects
 			(font
@@
 	(symbol
 		(lib_id "power:GND")
-		(at 127 68.58 0)
+		(at 124.46 68.58 0)
 		(unit 1)
 		(exclude_from_sim no)
@@
 		(fields_autoplaced yes)
 		(property "Reference" "#PWR062"
-			(at 127 74.93 0)
+			(at 124.46 74.93 0)
 			(effects
 				(font
@@
 		)
 		(property "Value" "GND"
-			(at 127 73.66 0)
+			(at 124.46 73.66 0)
 			(effects
 				(font
@@
 		)
 		(property "Footprint" ""
-			(at 127 68.58 0)
+			(at 124.46 68.58 0)
 			(effects
 				(font
@@
 		)
 		(property "Datasheet" ""
-			(at 127 68.58 0)
+			(at 124.46 68.58 0)
 			(effects
 				(font
@@
 		)
 		(property "Description" "Power symbol creates a global label with name \"GND\" , ground"
-			(at 127 68.58 0)
+			(at 124.46 68.58 0)
 			(effects
 				(font
@@
 			)
 		)
-		(property "Value" "57.6k"
+		(property "Value" "76.8k"
 			(at 228.6 77.4699 0)
 			(effects
@@
 			)
 		)
-		(property "Value" "76.8k"
+		(property "Value" "57.6k"
 			(at 243.84 77.4699 0)
 			(effects
@@
 	(symbol
 		(lib_id "Device:C_Small")
-		(at 127 66.04 0)
+		(at 124.46 66.04 0)
 		(unit 1)
 		(exclude_from_sim no)
@@
 		(dnp no)
 		(property "Reference" "C10"
-			(at 129.54 64.7762 0)
+			(at 127 64.7762 0)
 			(effects
 				(font
@@
 		)
 		(property "Value" "100n"
-			(at 129.54 67.3162 0)
+			(at 127 67.3162 0)
 			(effects
 				(font
@@
 		)
 		(property "Footprint" "Capacitor_SMD:C_0603_1608Metric"
-			(at 127 66.04 0)
+			(at 124.46 66.04 0)
 			(effects
 				(font
@@
 		)
 		(property "Datasheet" "~"
-			(at 127 66.04 0)
+			(at 124.46 66.04 0)
 			(effects
 				(font
@@
 		)
 		(property "Description" "Unpolarized capacitor, small symbol"
-			(at 127 66.04 0)
+			(at 124.46 66.04 0)
 			(effects
 				(font
@@
 			)
 		)
-		(property "Value" "700k"
+		(property "Value" "500k"
 			(at 203.2 77.4699 0)
 			(effects
@@
 			)
 		)
-		(property "Value" "26.1k"
+		(property "Value" "44.2k"
 			(at 243.84 82.5499 0)
 			(effects
@@
 			)
 		)
-		(property "Value" "500k"
+		(property "Value" "700k"
 			(at 193.04 77.4699 0)
 			(effects
@@
 	)
 	(symbol
-		(lib_id "power:GND")
-		(at 39.37 76.2 0)
-		(mirror y)
-		(unit 1)
-		(exclude_from_sim no)
-		(in_bom yes)
-		(on_board yes)
-		(dnp no)
-		(fields_autoplaced yes)
-		(property "Reference" "#PWR054"
-			(at 39.37 82.55 0)
-			(effects
-				(font
-					(size 1.27 1.27)
-				)
-				(hide yes)
-			)
-		)
-		(property "Value" "GND"
-			(at 39.37 81.28 0)
-			(effects
-				(font
-					(size 1.27 1.27)
-				)
-			)
-		)
-		(property "Footprint" ""
-			(at 39.37 76.2 0)
-			(effects
-				(font
-					(size 1.27 1.27)
-				)
-				(hide yes)
-			)
-		)
-		(property "Datasheet" ""
-			(at 39.37 76.2 0)
-			(effects
-				(font
-					(size 1.27 1.27)
-				)
-				(hide yes)
-			)
-		)
-		(property "Description" "Power symbol creates a global label with name \"GND\" , ground"
-			(at 39.37 76.2 0)
-			(effects
-				(font
-					(size 1.27 1.27)
-				)
-				(hide yes)
-			)
-		)
-		(pin "1"
-		)
-		(instances
-			(project "powerdist"
-				(path "/d8b3361c-0c6a-4299-baf2-0b5966ddedfb/80ef8331-114c-4f92-a863-3bf968229e3d"
-					(reference "#PWR054")
-					(unit 1)
-				)
-				(path "/d8b3361c-0c6a-4299-baf2-0b5966ddedfb/c1d41094-c001-4e3e-876f-0ad999dbbb80"
-					(reference "#PWR092")
-					(unit 1)
-				)
-				(path "/d8b3361c-0c6a-4299-baf2-0b5966ddedfb/ee142fce-035e-4426-8777-c2a0029f9d07"
-					(reference "#PWR073")
-					(unit 1)
-				)
-			)
-		)
-	)
-	(symbol
 		(lib_id "Device:C_Small")
 		(at 88.9 74.93 0)
@@
 	)
 	(symbol
-		(lib_id "Device:R_Small_US")
-		(at 39.37 73.66 0)
-		(mirror y)
-		(unit 1)
-		(exclude_from_sim no)
-		(in_bom yes)
-		(on_board yes)
-		(dnp no)
-		(property "Reference" "R16"
-			(at 36.83 72.3899 0)
-			(effects
-				(font
-					(size 1.27 1.27)
-				)
-				(justify left)
-			)
-		)
-		(property "Value" "100k"
-			(at 36.83 74.9299 0)
-			(effects
-				(font
-					(size 1.27 1.27)
-				)
-				(justify left)
-			)
-		)
-		(property "Footprint" "Resistor_SMD:R_0603_1608Metric"
-			(at 39.37 73.66 0)
-			(effects
-				(font
-					(size 1.27 1.27)
-				)
-				(hide yes)
-			)
-		)
-		(property "Datasheet" "~"
-			(at 39.37 73.66 0)
-			(effects
-				(font
-					(size 1.27 1.27)
-				)
-				(hide yes)
-			)
-		)
-		(property "Description" "Resistor, small US symbol"
-			(at 39.37 73.66 0)
-			(effects
-				(font
-					(size 1.27 1.27)
-				)
-				(hide yes)
-			)
-		)
-		(pin "1"
-		)
-		(pin "2"
-		)
-		(instances
-			(project "powerdist"
-				(path "/d8b3361c-0c6a-4299-baf2-0b5966ddedfb/80ef8331-114c-4f92-a863-3bf968229e3d"
-					(reference "R16")
-					(unit 1)
-				)
-				(path "/d8b3361c-0c6a-4299-baf2-0b5966ddedfb/c1d41094-c001-4e3e-876f-0ad999dbbb80"
-					(reference "R54")
-					(unit 1)
-				)
-				(path "/d8b3361c-0c6a-4299-baf2-0b5966ddedfb/ee142fce-035e-4426-8777-c2a0029f9d07"
-					(reference "R35")
-					(unit 1)
-				)
-			)
-		)
-	)
-	(symbol
 		(lib_id "Switch:SW_SPDT")
 		(at 195.58 67.31 270)
@@
 			)
 		)
-		(property "Value" "44.2k"
+		(property "Value" "26.1k"
 			(at 228.6 82.5499 0)
 			(effects

Commit message: local 31/10: PCB ordered
Parts:
- R13, R14, R15: value 895 -> 2k
- R17, R18: value 500k -> 100k
- R19: value 700k -> 500k
- R20: value 500k -> 698k
Changed lines of the file:
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@@
 		)
 	)
-	(text "4S"
+	(text "3S"
 		(exclude_from_sim no)
 		(at 200.66 81.026 0)
@@
 		)
 	)
-	(text "3S\n"
+	(text "4S\n"
 		(exclude_from_sim no)
 		(at 190.5 81.026 0)
@@
 			)
 		)
-		(property "Value" "500k"
+		(property "Value" "100k"
 			(at 123.19 81.2799 0)
 			(effects
@@
 			)
 		)
-		(property "Value" "500k"
+		(property "Value" "100k"
 			(at 123.19 86.3599 0)
 			(effects
@@
 			)
 		)
-		(property "Value" "895"
+		(property "Value" "2k"
 			(at 35.56 57.15 90)
 			(effects
@@
 			)
 		)
-		(property "Value" "500k"
+		(property "Value" "698k"
 			(at 203.2 77.4699 0)
 			(effects
@@
 			)
 		)
-		(property "Value" "895"
+		(property "Value" "2k"
 			(at 35.56 48.26 90)
 			(effects
@@
 			)
 		)
-		(property "Value" "700k"
+		(property "Value" "500k"
 			(at 193.04 77.4699 0)
 			(effects
@@
 			)
 		)
-		(property "Value" "895"
+		(property "Value" "2k"
 			(at 35.56 66.04 90)
 			(effects

Commit message: lab 06/12
Other:
- note added: "BAD CHARGE SETTING (PARALLEL RESISTORS)"
Changed lines of the file:
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@@
+		)
+	)
+	(text "BAD CHARGE SETTING (PARALLEL RESISTORS)"
+		(exclude_from_sim no)
+		(at 260.096 175.006 0)
+		(effects
+			(font
+				(size 1.27 1.27)
+			)
 		)
 	)
