File: powerdist/battprot_v0.2.kicad_sch (KiCad schematic)
At the start: 32 parts, among them Q23 L2N7002SLLT1G, Q24 IRF9388, Q3 IRF9388, Q6 L2N7002SLLT1G, SW3 SSSF021500, U2 BQ7791508PWR

Commit message: local 13/10
Parts:
- added R119: 10k, symbol Device:R_Small_US
- added TH3: 103AT-11, symbol Device:Thermistor_US
- renumbered C13 to C88, C14 to C89, C15 to C90, C16 to C91, C17 to C92, C18 to C93, C19 to C94, C20 to C95, C21 to C96, C22 to C97, D4 to D21, Q23 to Q19, Q24 to Q20, Q6 to Q21, Q3 to Q22, R22 to R111, R23 to R112, R24 to R113, R25 to R114, R26 to R115, R27 to R116, R28 to R117, R29 to R118, R30 to R120, R32 to R121, R31 to R122, R51 to R123, R2 to R124, R35 to R125, R36 to R126, SW3 to SW9, U2 to U9
Connections:
- net GND: now also TH3.1; no longer R115.1
- net TS: now also R119.2, TH3.2
- net Vtb: now also R119.1
- new net CELLGND: R115.1

Commit message: local 14/10
Parts:
- U9: footprint TSSOP24_4P4X7P8_THT_TEX -> powerdist:TSSOP24_4P4X7P8_THT_TEX
Changed lines of the file:
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@@
 		(dnp no)
 		(fields_autoplaced yes)
-		(property "Reference" "#FLG015"
+		(property "Reference" "#FLG023"
 			(at 279.4 160.655 0)
 			(effects
@@
 			(project "powerdist"
 				(path "/d8b3361c-0c6a-4299-baf2-0b5966ddedfb/754cc4f7-7309-49ec-a85a-88e49e6da610/0212c3ea-6f98-431b-bd03-36e6e092d236"
-					(reference "#FLG015")
-					(unit 1)
-				)
-				(path "/d8b3361c-0c6a-4299-baf2-0b5966ddedfb/754cc4f7-7309-49ec-a85a-88e49e6da610/1b151f5e-d113-49d8-a928-351d73068788"
-					(reference "#FLG06")
-					(unit 1)
-				)
-				(path "/d8b3361c-0c6a-4299-baf2-0b5966ddedfb/754cc4f7-7309-49ec-a85a-88e49e6da610/b47836f1-283b-4d17-ad51-d7ed8020bd0f"
-					(reference "#FLG014")
+					(reference "#FLG023")
+					(unit 1)
+				)
+				(path "/d8b3361c-0c6a-4299-baf2-0b5966ddedfb/754cc4f7-7309-49ec-a85a-88e49e6da610/1b151f5e-d113-49d8-a928-351d73068788"
+					(reference "#FLG09")
+					(unit 1)
+				)
+				(path "/d8b3361c-0c6a-4299-baf2-0b5966ddedfb/754cc4f7-7309-49ec-a85a-88e49e6da610/b47836f1-283b-4d17-ad51-d7ed8020bd0f"
+					(reference "#FLG022")
 					(unit 1)
 				)
@@
 			)
 		)
-		(property "Footprint" "TSSOP24_4P4X7P8_THT_TEX"
+		(property "Footprint" "powerdist:TSSOP24_4P4X7P8_THT_TEX"
 			(at 172.212 112.776 0)
 			(effects

Commit message: local 19/10
Parts:
- renumbered C88 to C100, C89 to C101, C90 to C102, C91 to C103, C92 to C104, C93 to C105, C94 to C106, C95 to C107, C96 to C108, C97 to C109
Changed lines of the file:
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@@
 		(on_board yes)
 		(dnp no)
-		(property "Reference" "C91"
+		(property "Reference" "C103"
 			(at 39.37 35.5662 0)
 			(effects
@@
 			(project ""
 				(path "/d8b3361c-0c6a-4299-baf2-0b5966ddedfb/754cc4f7-7309-49ec-a85a-88e49e6da610/0212c3ea-6f98-431b-bd03-36e6e092d236"
-					(reference "C91")
+					(reference "C103")
 					(unit 1)
 				)
 				(path "/d8b3361c-0c6a-4299-baf2-0b5966ddedfb/754cc4f7-7309-49ec-a85a-88e49e6da610/1b151f5e-d113-49d8-a928-351d73068788"
-					(reference "C18")
+					(reference "C22")
 					(unit 1)
 				)
 				(path "/d8b3361c-0c6a-4299-baf2-0b5966ddedfb/754cc4f7-7309-49ec-a85a-88e49e6da610/b47836f1-283b-4d17-ad51-d7ed8020bd0f"
-					(reference "C81")
+					(reference "C93")
 					(unit 1)
 				)
@@
 		(on_board yes)
 		(dnp no)
-		(property "Reference" "C90"
+		(property "Reference" "C102"
 			(at 38.1 59.6962 0)
 			(effects
@@
 			(project ""
 				(path "/d8b3361c-0c6a-4299-baf2-0b5966ddedfb/754cc4f7-7309-49ec-a85a-88e49e6da610/0212c3ea-6f98-431b-bd03-36e6e092d236"
-					(reference "C90")
+					(reference "C102")
 					(unit 1)
 				)
 				(path "/d8b3361c-0c6a-4299-baf2-0b5966ddedfb/754cc4f7-7309-49ec-a85a-88e49e6da610/1b151f5e-d113-49d8-a928-351d73068788"
-					(reference "C17")
+					(reference "C21")
 					(unit 1)
 				)
 				(path "/d8b3361c-0c6a-4299-baf2-0b5966ddedfb/754cc4f7-7309-49ec-a85a-88e49e6da610/b47836f1-283b-4d17-ad51-d7ed8020bd0f"
-					(reference "C80")
+					(reference "C92")
 					(unit 1)
 				)
@@
 		(on_board yes)
 		(dnp no)
-		(property "Reference" "C94"
+		(property "Reference" "C106"
 			(at 78.7462 52.07 0)
 			(effects
@@
 			(project ""
 				(path "/d8b3361c-0c6a-4299-baf2-0b5966ddedfb/754cc4f7-7309-49ec-a85a-88e49e6da610/0212c3ea-6f98-431b-bd03-36e6e092d236"
-					(reference "C94")
+					(reference "C106")
 					(unit 1)
 				)
 				(path "/d8b3361c-0c6a-4299-baf2-0b5966ddedfb/754cc4f7-7309-49ec-a85a-88e49e6da610/1b151f5e-d113-49d8-a928-351d73068788"
-					(reference "C21")
+					(reference "C25")
 					(unit 1)
 				)
 				(path "/d8b3361c-0c6a-4299-baf2-0b5966ddedfb/754cc4f7-7309-49ec-a85a-88e49e6da610/b47836f1-283b-4d17-ad51-d7ed8020bd0f"
-					(reference "C84")
+					(reference "C96")
 					(unit 1)
 				)
@@
 		(on_board yes)
 		(dnp no)
-		(property "Reference" "C93"
+		(property "Reference" "C105"
 			(at 73.6538 46.99 0)
 			(effects
@@
 			(project ""
 				(path "/d8b3361c-0c6a-4299-baf2-0b5966ddedfb/754cc4f7-7309-49ec-a85a-88e49e6da610/0212c3ea-6f98-431b-bd03-36e6e092d236"
-					(reference "C93")
+					(reference "C105")
 					(unit 1)
 				)
 				(path "/d8b3361c-0c6a-4299-baf2-0b5966ddedfb/754cc4f7-7309-49ec-a85a-88e49e6da610/1b151f5e-d113-49d8-a928-351d73068788"
-					(reference "C20")
+					(reference "C24")
 					(unit 1)
 				)
 				(path "/d8b3361c-0c6a-4299-baf2-0b5966ddedfb/754cc4f7-7309-49ec-a85a-88e49e6da610/b47836f1-283b-4d17-ad51-d7ed8020bd0f"
-					(reference "C83")
+					(reference "C95")
 					(unit 1)
 				)
@@
 		(on_board yes)
 		(dnp no)
-		(property "Reference" "C89"
+		(property "Reference" "C101"
 			(at 38.1 44.4562 0)
 			(effects
@@
 			(project ""
 				(path "/d8b3361c-0c6a-4299-baf2-0b5966ddedfb/754cc4f7-7309-49ec-a85a-88e49e6da610/0212c3ea-6f98-431b-bd03-36e6e092d236"
-					(reference "C89")
+					(reference "C101")
 					(unit 1)
 				)
 				(path "/d8b3361c-0c6a-4299-baf2-0b5966ddedfb/754cc4f7-7309-49ec-a85a-88e49e6da610/1b151f5e-d113-49d8-a928-351d73068788"
-					(reference "C16")
+					(reference "C20")
 					(unit 1)
 				)
 				(path "/d8b3361c-0c6a-4299-baf2-0b5966ddedfb/754cc4f7-7309-49ec-a85a-88e49e6da610/b47836f1-283b-4d17-ad51-d7ed8020bd0f"
-					(reference "C79")
+					(reference "C91")
 					(unit 1)
 				)
@@
 		(on_board yes)
 		(dnp no)
-		(property "Reference" "C92"
+		(property "Reference" "C104"
 			(at 39.37 52.0762 0)
 			(effects
@@
 			(project ""
 				(path "/d8b3361c-0c6a-4299-baf2-0b5966ddedfb/754cc4f7-7309-49ec-a85a-88e49e6da610/0212c3ea-6f98-431b-bd03-36e6e092d236"
-					(reference "C92")
+					(reference "C104")
 					(unit 1)
 				)
 				(path "/d8b3361c-0c6a-4299-baf2-0b5966ddedfb/754cc4f7-7309-49ec-a85a-88e49e6da610/1b151f5e-d113-49d8-a928-351d73068788"
-					(reference "C19")
+					(reference "C23")
 					(unit 1)
 				)
 				(path "/d8b3361c-0c6a-4299-baf2-0b5966ddedfb/754cc4f7-7309-49ec-a85a-88e49e6da610/b47836f1-283b-4d17-ad51-d7ed8020bd0f"
-					(reference "C82")
+					(reference "C94")
 					(unit 1)
 				)
@@
 		(on_board yes)
 		(dnp no)
-		(property "Reference" "C97"
+		(property "Reference" "C109"
 			(at 139.7 81.2862 0)
 			(effects
@@
 			(project ""
 				(path "/d8b3361c-0c6a-4299-baf2-0b5966ddedfb/754cc4f7-7309-49ec-a85a-88e49e6da610/0212c3ea-6f98-431b-bd03-36e6e092d236"
-					(reference "C97")
+					(reference "C109")
 					(unit 1)
 				)
 				(path "/d8b3361c-0c6a-4299-baf2-0b5966ddedfb/754cc4f7-7309-49ec-a85a-88e49e6da610/1b151f5e-d113-49d8-a928-351d73068788"
-					(reference "C24")
+					(reference "C28")
 					(unit 1)
 				)
 				(path "/d8b3361c-0c6a-4299-baf2-0b5966ddedfb/754cc4f7-7309-49ec-a85a-88e49e6da610/b47836f1-283b-4d17-ad51-d7ed8020bd0f"
-					(reference "C87")
+					(reference "C99")
 					(unit 1)
 				)
@@
 		(on_board yes)
 		(dnp no)
-		(property "Reference" "C96"
+		(property "Reference" "C108"
 			(at 130.81 78.7462 0)
 			(effects
@@
 			(project ""
 				(path "/d8b3361c-0c6a-4299-baf2-0b5966ddedfb/754cc4f7-7309-49ec-a85a-88e49e6da610/0212c3ea-6f98-431b-bd03-36e6e092d236"
-					(reference "C96")
+					(reference "C108")
 					(unit 1)
 				)
 				(path "/d8b3361c-0c6a-4299-baf2-0b5966ddedfb/754cc4f7-7309-49ec-a85a-88e49e6da610/1b151f5e-d113-49d8-a928-351d73068788"
-					(reference "C23")
+					(reference "C27")
 					(unit 1)
 				)
 				(path "/d8b3361c-0c6a-4299-baf2-0b5966ddedfb/754cc4f7-7309-49ec-a85a-88e49e6da610/b47836f1-283b-4d17-ad51-d7ed8020bd0f"
-					(reference "C86")
+					(reference "C98")
 					(unit 1)
 				)
@@
 		(on_board yes)
 		(dnp no)
-		(property "Reference" "C88"
+		(property "Reference" "C100"
 			(at 38.1 26.6762 0)
 			(effects
@@
 			(project ""
 				(path "/d8b3361c-0c6a-4299-baf2-0b5966ddedfb/754cc4f7-7309-49ec-a85a-88e49e6da610/0212c3ea-6f98-431b-bd03-36e6e092d236"
-					(reference "C88")
+					(reference "C100")
 					(unit 1)
 				)
 				(path "/d8b3361c-0c6a-4299-baf2-0b5966ddedfb/754cc4f7-7309-49ec-a85a-88e49e6da610/1b151f5e-d113-49d8-a928-351d73068788"
-					(reference "C15")
+					(reference "C19")
 					(unit 1)
 				)
 				(path "/d8b3361c-0c6a-4299-baf2-0b5966ddedfb/754cc4f7-7309-49ec-a85a-88e49e6da610/b47836f1-283b-4d17-ad51-d7ed8020bd0f"
-					(reference "C78")
+					(reference "C90")
 					(unit 1)
 				)
@@
 		(on_board yes)
 		(dnp no)
-		(property "Reference" "C95"
+		(property "Reference" "C107"
 			(at 88.8938 46.99 0)
 			(effects
@@
 			(project ""
 				(path "/d8b3361c-0c6a-4299-baf2-0b5966ddedfb/754cc4f7-7309-49ec-a85a-88e49e6da610/0212c3ea-6f98-431b-bd03-36e6e092d236"
-					(reference "C95")
+					(reference "C107")
 					(unit 1)
 				)
 				(path "/d8b3361c-0c6a-4299-baf2-0b5966ddedfb/754cc4f7-7309-49ec-a85a-88e49e6da610/1b151f5e-d113-49d8-a928-351d73068788"
-					(reference "C22")
+					(reference "C26")
 					(unit 1)
 				)
 				(path "/d8b3361c-0c6a-4299-baf2-0b5966ddedfb/754cc4f7-7309-49ec-a85a-88e49e6da610/b47836f1-283b-4d17-ad51-d7ed8020bd0f"
-					(reference "C85")
+					(reference "C97")
 					(unit 1)
 				)

Commit message: lab 20/10
Parts:
- Q23: renamed from Q20; value IRF9388 -> SIS412DN
- Q25: renamed from Q22; value IRF9388 -> SIS412DN
- renumbered D21 to D23, Q19 to Q22, Q21 to Q24, R111 to R114, R112 to R115, R113 to R116, R114 to R117, R115 to R118, R116 to R119, R117 to R120, R118 to R121, R119 to R122, R120 to R123, R121 to R124, R122 to R125, R123 to R126, R124 to R127, R125 to R128, R126 to R129

Commit message: lab 21/10
Parts:
- D24: renamed from D23; footprint (none) -> Package_TO_SOT_SMD:TO-277A
- R114, R115, R116, R117, R118, R119, R120, R121, R122, R123, R124, R125, R126, R127, R128, R129: footprint (none) -> Resistor_SMD:R_0603_1608Metric
- SW9: value SSSF021500 -> JS202011CQN; footprint (none) -> Button_Switch_THT:SW_CK_JS202011CQN_DPDT_Straight
- TH3: footprint (none) -> Resistor_THT:R_Box_L8.4mm_W2.5mm_P5.08mm
Changed lines of the file:
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@@
 			)
 		)
-		(property "Footprint" ""
+		(property "Footprint" "Resistor_SMD:R_0603_1608Metric"
 			(at 76.2 54.61 0)
 			(effects
@@
 			)
 		)
-		(property "Footprint" ""
+		(property "Footprint" "Resistor_SMD:R_0603_1608Metric"
 			(at 80.01 59.69 0)
 			(effects
@@
 			)
 		)
-		(property "Footprint" ""
+		(property "Footprint" "Resistor_SMD:R_0603_1608Metric"
 			(at 231.14 27.94 0)
 			(effects
@@
 			)
 		)
-		(property "Footprint" ""
+		(property "Footprint" "Resistor_SMD:R_0603_1608Metric"
 			(at 265.43 43.18 0)
 			(effects
@@
 			)
 		)
-		(property "Footprint" ""
+		(property "Footprint" "Resistor_SMD:R_0603_1608Metric"
 			(at 30.48 64.77 0)
 			(effects
@@
 			)
 		)
-		(property "Footprint" ""
+		(property "Footprint" "Resistor_SMD:R_0603_1608Metric"
 			(at 27.94 49.53 0)
 			(effects
@@
 			)
 		)
-		(property "Footprint" ""
+		(property "Footprint" "Resistor_SMD:R_0603_1608Metric"
 			(at 129.54 76.2 0)
 			(effects
@@
 			)
 		)
-		(property "Value" "SSSF021500"
+		(property "Value" "JS202011CQN"
 			(at 76.2 20.32 0)
 			(effects
@@
 			)
 		)
-		(property "Footprint" ""
+		(property "Footprint" "Button_Switch_THT:SW_CK_JS202011CQN_DPDT_Straight"
 			(at 76.2 26.67 0)
 			(effects
@@
 			)
 		)
-		(property "Footprint" ""
+		(property "Footprint" "Resistor_SMD:R_0603_1608Metric"
 			(at 265.43 27.94 0)
 			(effects
@@
 			)
 		)
-		(property "Footprint" ""
+		(property "Footprint" "Resistor_SMD:R_0603_1608Metric"
 			(at 83.82 54.61 0)
 			(effects
@@
 			)
 		)
-		(property "Footprint" ""
+		(property "Footprint" "Resistor_SMD:R_0603_1608Metric"
 			(at 27.94 22.86 0)
 			(effects
@@
 			)
 		)
-		(property "Footprint" ""
+		(property "Footprint" "Resistor_SMD:R_0603_1608Metric"
 			(at 27.94 31.75 0)
 			(effects
@@
 			)
 		)
-		(property "Footprint" ""
+		(property "Footprint" "Resistor_SMD:R_0603_1608Metric"
 			(at 196.85 95.25 0)
 			(effects
@@
 			)
 		)
-		(property "Value" "SSSF021500"
+		(property "Value" "JS202011CQN"
 			(at 52.07 19.05 0)
 			(effects
@@
 			)
 		)
-		(property "Footprint" ""
+		(property "Footprint" "Button_Switch_THT:SW_CK_JS202011CQN_DPDT_Straight"
 			(at 52.07 25.4 0)
 			(effects
@@
 			)
 		)
-		(property "Footprint" ""
+		(property "Footprint" "Resistor_THT:R_Box_L8.4mm_W2.5mm_P5.08mm"
 			(at 99.06 27.94 0)
 			(effects
@@
 			)
 		)
-		(property "Footprint" ""
+		(property "Footprint" "Resistor_SMD:R_0603_1608Metric"
 			(at 199.39 82.55 0)
 			(effects
@@
 		(on_board yes)
 		(dnp no)
-		(property "Reference" "D23"
+		(property "Reference" "D24"
 			(at 244.094 30.48 0)
 			(effects
@@
 			)
 		)
-		(property "Footprint" ""
+		(property "Footprint" "Package_TO_SOT_SMD:TO-277A"
 			(at 243.84 24.13 90)
 			(effects
@@
 			(project ""
 				(path "/d8b3361c-0c6a-4299-baf2-0b5966ddedfb/754cc4f7-7309-49ec-a85a-88e49e6da610/0212c3ea-6f98-431b-bd03-36e6e092d236"
-					(reference "D23")
+					(reference "D24")
 					(unit 1)
 				)
 				(path "/d8b3361c-0c6a-4299-baf2-0b5966ddedfb/754cc4f7-7309-49ec-a85a-88e49e6da610/1b151f5e-d113-49d8-a928-351d73068788"
-					(reference "D10")
+					(reference "D11")
 					(unit 1)
 				)
 				(path "/d8b3361c-0c6a-4299-baf2-0b5966ddedfb/754cc4f7-7309-49ec-a85a-88e49e6da610/b47836f1-283b-4d17-ad51-d7ed8020bd0f"
-					(reference "D22")
+					(reference "D23")
 					(unit 1)
 				)
@@
 			)
 		)
-		(property "Footprint" ""
+		(property "Footprint" "Resistor_SMD:R_0603_1608Metric"
 			(at 27.94 40.64 0)
 			(effects
@@
 			)
 		)
-		(property "Footprint" ""
+		(property "Footprint" "Resistor_SMD:R_0603_1608Metric"
 			(at 99.06 21.59 0)
 			(effects
@@
 			)
 		)
-		(property "Footprint" ""
+		(property "Footprint" "Resistor_SMD:R_0603_1608Metric"
 			(at 231.14 43.18 0)
 			(effects

Commit message: lab 23/10
Parts:
- C100, C101, C102, C103, C104, C105, C106, C107, C108, C109: footprint (none) -> Capacitor_SMD:C_0603_1608Metric
- D24: symbol Device:D_Schottky_Small_Filled -> D_Schottky_AAK_Parallel_Small_Filled:D_Schottky_AAK
- Q22, Q24: footprint (none) -> Package_TO_SOT_SMD:SOT-23
- Q23, Q25: footprint (none) -> Package_SO:Vishay_PowerPAK_1212-8_Single; symbol Simulation_SPICE:PMOS -> Transistor_FET:SiS454DN
Connections:
- net +BATT: now also D24.3 (K); no longer D24.1 (K)
- net Vbatt: now also Q23.1 (S), Q23.2 (S), Q25.5 (D); no longer Q25.1 (D)
- net Vin: now also Q25.1 (S), Q25.2 (S)
- net at Q22.1 (D), R126.2: now also Q23.4 (G); no longer Q23.2 (G)
- net at Q24.1 (D), R128.2: now also Q25.4 (G); no longer Q25.2 (G)
- net at D24.2 (A): now also D24.1 (A), Q23.5 (D); no longer Q23.1 (D)
Other:
- moved on the sheet: Q22, Q23, R126, R127

Commit message: local 26/10
Parts:
- R75: renamed from R120; footprint Resistor_SMD:R_0603_1608Metric -> Resistor_SMD:R_1206_3216Metric
- TH1: renamed from TH3; footprint Resistor_THT:R_Box_L8.4mm_W2.5mm_P5.08mm -> Connector_JST:JST_XH_B2B-XH-AM_1x02_P2.50mm_Vertical
- renumbered C100 to C49, C101 to C50, C102 to C51, C103 to C52, C104 to C53, C105 to C54, C106 to C55, C107 to C56, C108 to C57, C109 to C58, Q22 to Q15, Q23 to Q16, Q24 to Q17, Q25 to Q18, R114 to R69, R115 to R70, R116 to R71, R117 to R72, R118 to R73, R119 to R74, R121 to R76, R122 to R77, R123 to R78, R124 to R79, R125 to R80, R126 to R81, R127 to R82, R128 to R83, R129 to R84, SW9 to SW7, U9 to U4
Connections:
- net PSRN: now also C55.2, C56.2, R76.2; no longer C54.1, C55.1, R74.1
- net PSRP: now also C54.1, C55.1, R74.1; no longer C55.2, C56.2, R76.2
- net +BATT renamed Vout

Commit message: local 28/10
Parts:
- Q15, Q17: symbol Simulation_SPICE:NMOS -> Transistor_FET:2N7002
Connections:
- net CHG: now also Q17.1 (G); no longer Q17.2 (G)
- net DSG: now also Q15.1 (G); no longer Q15.2 (G)
- net GND: now also Q15.2 (S), Q17.2 (S); no longer Q15.3 (S), Q17.3 (S)
- net at Q16.4 (G), R81.2: now also Q15.3 (D); no longer Q15.1 (D)
- net at Q18.4 (G), R83.2: now also Q17.3 (D); no longer Q17.1 (D)
Changed lines of the file:
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@@
 	)
 	(symbol
-		(lib_id "Simulation_SPICE:NMOS")
+		(lib_id "Transistor_FET:2N7002")
 		(at 232.41 36.83 0)
 		(unit 1)
@@
 		)
 		(property "Footprint" "Package_TO_SOT_SMD:SOT-23"
-			(at 237.49 34.29 0)
-			(effects
-				(font
-					(size 1.27 1.27)
-				)
-				(hide yes)
-			)
-		)
-		(property "Datasheet" "https://ngspice.sourceforge.io/docs/ngspice-html-manual/manual.xhtml#cha_MOSFETs"
-			(at 232.41 49.53 0)
-			(effects
-				(font
-					(size 1.27 1.27)
-				)
-				(hide yes)
-			)
-		)
-		(property "Description" "N-MOSFET transistor, drain/source/gate"
+			(at 237.49 38.735 0)
+			(effects
+				(font
+					(size 1.27 1.27)
+					(italic yes)
+				)
+				(justify left)
+				(hide yes)
+			)
+		)
+		(property "Datasheet" "https://www.onsemi.com/pub/Collateral/NDS7002A-D.PDF"
+			(at 237.49 40.64 0)
+			(effects
+				(font
+					(size 1.27 1.27)
+				)
+				(justify left)
+				(hide yes)
+			)
+		)
+		(property "Description" "0.115A Id, 60V Vds, N-Channel MOSFET, SOT-23"
 			(at 232.41 36.83 0)
 			(effects
@@
 	)
 	(symbol
-		(lib_id "Simulation_SPICE:NMOS")
+		(lib_id "Transistor_FET:2N7002")
 		(at 267.97 36.83 0)
 		(unit 1)
@@
 		)
 		(property "Footprint" "Package_TO_SOT_SMD:SOT-23"
-			(at 273.05 34.29 0)
-			(effects
-				(font
-					(size 1.27 1.27)
-				)
-				(hide yes)
-			)
-		)
-		(property "Datasheet" "https://ngspice.sourceforge.io/docs/ngspice-html-manual/manual.xhtml#cha_MOSFETs"
-			(at 267.97 49.53 0)
-			(effects
-				(font
-					(size 1.27 1.27)
-				)
-				(hide yes)
-			)
-		)
-		(property "Description" "N-MOSFET transistor, drain/source/gate"
+			(at 273.05 38.735 0)
+			(effects
+				(font
+					(size 1.27 1.27)
+					(italic yes)
+				)
+				(justify left)
+				(hide yes)
+			)
+		)
+		(property "Datasheet" "https://www.onsemi.com/pub/Collateral/NDS7002A-D.PDF"
+			(at 273.05 40.64 0)
+			(effects
+				(font
+					(size 1.27 1.27)
+				)
+				(justify left)
+				(hide yes)
+			)
+		)
+		(property "Description" "0.115A Id, 60V Vds, N-Channel MOSFET, SOT-23"
 			(at 267.97 36.83 0)
 			(effects
