File: powerdist/battprot_v0.2.kicad_sch (KiCad schematic)
At the start: 34 parts, among them Q15 L2N7002SLLT1G, Q16 SIS412DN, Q17 L2N7002SLLT1G, Q18 SIS412DN, SW7 JS202011CQN, U4 BQ7791508PWR

Commit message: lab 27/11
Other:
- note added: "STUPID SW7 NO CELL BALANCING (or 1k Rin) INCORRECT HIGH-SIDE LOGIC"
Changed lines of the file:
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@@
+		)
+	)
+	(text "STUPID SW7\nNO CELL BALANCING (or 1k Rin)\nINCORRECT HIGH-SIDE LOGIC"
+		(exclude_from_sim no)
+		(at 261.366 176.53 0)
+		(effects
+			(font
+				(size 1.27 1.27)
+			)
 		)
 	)
