File: powerdist/powerdist.kicad_pcb (KiCad board)
At the start: 2 copper layers, 370 parts, among them J1 Conn_01x02_Socket, J10 Conn_01x02_Pin, J11 Conn_01x02_Pin, J12 Conn_01x02_Pin, J13 Conn_01x02_Pin, J2 Conn_01x02_Socket, J3 Conn_01x02_Socket, J3 Conn_01x04_Socket, J4 Conn_01x04_Pin, J5 Conn_01x02_Socket, J6 Conn_01x02_Socket, J7 Conn_01x02_Socket, J8 Conn_01x02_Socket, J9 Conn_01x04_Socket, Q1 SI4178DY, Q10 SIS412DN, Q11 SIS412DN, Q12 SIS412DN, Q13 SIS412DN, Q14 SIS412DN, Q15 L2N7002SLLT1G, Q16 SIS412DN, Q17 L2N7002SLLT1G, Q18 SIS412DN, Q19 L2N7002SLLT1G, Q2 SI4178DY, Q20 SIS412DN, Q21 L2N7002SLLT1G, Q22 SIS412DN, Q23 L2N7002SLLT1G, Q24 SIS412DN, Q25 L2N7002SLLT1G, Q26 SIS412DN, Q27 CSD18514Q5A, Q28 CSD18514Q5A, Q29 CSD18514Q5A, Q3 SI4178DY, Q30 CSD18514Q5A, Q4 SI4178DY, Q5 DMN2056U, Q6 DMN2056U, Q7 DMN2056U, Q8 DMN2056U, Q9 SIS412DN, SW1 OS102011M, SW2 JS202011CQN, SW3 OS102011M, SW4 JS202011CQN, SW5 OS102011M, SW6 JS202011CQN, SW7 JS202011CQN, SW8 JS202011CQN, SW9 JS202011CQN, U1 BQ24610, U10 TPS56637RPAR, U11 TPS56637RPAR, U12 ACS724LLCTR-10AU, U13 ACS724LLCTR-10AU, U14 ACS724LLCTR-10AU, U15 ACS724LLCTR-10AU, U16 ADS1119IPWR, U2 BQ24610, U3 BQ24610, U4 BQ7791508PWR, U5 BQ7791508PWR, U6 BQ7791508PWR, U7 LM5176PWP, U8 ACS724LLCTR-10AU, U9 ADS1119IPWR

Commit message: lab 27/10
Parts:
- removed the J3 at (242.8, 51.4)
- R128, R26, R45, R64: footprint Resistor_SMD:R_0603_1608Metric -> Resistor_SMD:R_1206_3216Metric
- moved R9 66.6 mm to (101.4, 146.0)
- moved D6 57.1 mm to (107.1, 145.7)
- moved D7 54.6 mm to (183.8, 78.9)
- moved R5 50.1 mm to (179.5, 65.3)
- moved R8 36.8 mm to (103.6, 102.0)
- moved SW1 34.2 mm to (95.3, 78.2)
- moved Q10 27.9 mm to (100.4, 40.1), turned to -90 degrees
- moved C4 27.6 mm to (110.9, 36.8), turned to 180 degrees
- moved D5 26.8 mm to (108.2, 102.5)
- moved L3 25.7 mm to (89.4, 42.3), turned to 180 degrees
- moved C18 25.1 mm to (75.9, 40.8), turned to 90 degrees
- moved R12 23.6 mm to (114.7, 36.8), turned to 180 degrees
- moved C12 23.1 mm to (105.7, 42.3), turned to 90 degrees
- moved C17 22.9 mm to (73.6, 40.8), turned to 90 degrees
- moved R26 22.2 mm to (79.4, 42.3), turned to 180 degrees
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Connections:
- C10 pad 1: /battcharger3S1/CSRN -> /battcharger4S/CSRN
- C13 pad 1: /battcharger3S1/CSRN -> /battcharger4S/CSRN
- C13 pad 2: /battcharger3S1/Vfb -> /battcharger4S/Vfb
- C14 pad 1: /battcharger3S1/BTST -> /battcharger4S/BTST
- C14 pad 2: /battcharger3S1/PH -> /battcharger4S/PH
- C15 pad 1: /battcharger3S1/CSRN -> /battcharger4S/CSRN
- C16 pad 1: /battcharger3S1/CSRN -> /battcharger4S/CSRN
- C17 pad 1: /battcharger3S1/CSRN -> /battcharger4S/CSRN
- C18 pad 1: /battcharger3S1/CSRN -> /battcharger4S/CSRN
- C21 pad 1: /battcharger3S2/Vref -> /battcharger3S1/Vref
- C23 pad 1: /battcharger3S2/REGN -> /battcharger3S1/REGN
- C24 pad 1: /battcharger3S2/CSRP -> /battcharger3S1/CSRP
- C24 pad 2: /battcharger3S2/CSRN -> /battcharger3S1/CSRN
- C25 pad 1: /battcharger3S2/CSRN -> /battcharger3S1/CSRN
- C28 pad 1: /battcharger3S2/CSRN -> /battcharger3S1/CSRN
- C28 pad 2: /battcharger3S2/Vfb -> /battcharger3S1/Vfb
- C29 pad 1: /battcharger3S2/BTST -> /battcharger3S1/BTST
- C29 pad 2: /battcharger3S2/PH -> /battcharger3S1/PH
- C30 pad 1: /battcharger3S2/CSRN -> /battcharger3S1/CSRN
- C31 pad 1: /battcharger3S2/CSRN -> /battcharger3S1/CSRN
- C32 pad 1: /battcharger3S2/CSRN -> /battcharger3S1/CSRN
- C33 pad 1: /battcharger3S2/CSRN -> /battcharger3S1/CSRN
- C36 pad 1: /battcharger4S/Vref -> /battcharger3S2/Vref
- C38 pad 1: /battcharger4S/REGN -> /battcharger3S2/REGN
- C39 pad 1: /battcharger4S/CSRP -> /battcharger3S2/CSRP
- C39 pad 2: /battcharger4S/CSRN -> /battcharger3S2/CSRN
- C40 pad 1: /battcharger4S/CSRN -> /battcharger3S2/CSRN
- C43 pad 1: /battcharger4S/CSRN -> /battcharger3S2/CSRN
- C43 pad 2: /battcharger4S/Vfb -> /battcharger3S2/Vfb
- C44 pad 1: /battcharger4S/BTST -> /battcharger3S2/BTST
- C44 pad 2: /battcharger4S/PH -> /battcharger3S2/PH
- C45 pad 1: /battcharger4S/CSRN -> /battcharger3S2/CSRN
- C46 pad 1: /battcharger4S/CSRN -> /battcharger3S2/CSRN
- C47 pad 1: /battcharger4S/CSRN -> /battcharger3S2/CSRN
- C48 pad 1: /battcharger4S/CSRN -> /battcharger3S2/CSRN
- C6 pad 1: /battcharger3S1/Vref -> /battcharger4S/Vref
- C8 pad 1: /battcharger3S1/REGN -> /battcharger4S/REGN
- C9 pad 1: /battcharger3S1/CSRP -> /battcharger4S/CSRP
- C9 pad 2: /battcharger3S1/CSRN -> /battcharger4S/CSRN
- D12 pad 1: /battcharger3S1/PG -> /battcharger4S/PG
- D13 pad 1: /CHG -> /CE
- D14 pad 1: /battcharger3S1/STAT2 -> /battcharger4S/STAT2
- D15 pad 1: /battcharger3S1/REGN -> /battcharger4S/REGN
- D15 pad 2: /battcharger3S1/REGN -> /battcharger4S/REGN
- D15 pad 3: /battcharger3S1/BTST -> /battcharger4S/BTST
- D16 pad 1: /battcharger3S2/PG -> /battcharger3S1/PG
- D18 pad 1: /battcharger3S2/STAT2 -> /battcharger3S1/STAT2
- D19 pad 1: /battcharger3S2/REGN -> /battcharger3S1/REGN
- D19 pad 2: /battcharger3S2/REGN -> /battcharger3S1/REGN
- D19 pad 3: /battcharger3S2/BTST -> /battcharger3S1/BTST
- D20 pad 1: /battcharger4S/PG -> /battcharger3S2/PG
- D21 pad 1: /CE -> /CHG
- D22 pad 1: /battcharger4S/STAT2 -> /battcharger3S2/STAT2
- D23 pad 1: /battcharger4S/REGN -> /battcharger3S2/REGN
- D23 pad 2: /battcharger4S/REGN -> /battcharger3S2/REGN
- D23 pad 3: /battcharger4S/BTST -> /battcharger3S2/BTST
- L3 pad 1: /battcharger3S1/PH -> /battcharger4S/PH
- L3 pad 2: /battcharger3S1/CSRP -> /battcharger4S/CSRP
- L4 pad 1: /battcharger3S2/PH -> /battcharger3S1/PH
- L4 pad 2: /battcharger3S2/CSRP -> /battcharger3S1/CSRP
- L5 pad 1: /battcharger4S/PH -> /battcharger3S2/PH
- L5 pad 2: /battcharger4S/CSRP -> /battcharger3S2/CSRP
- Q10 pad 4: /battcharger3S1/LODRV -> /battcharger4S/LODRV
- Q10 pad 5: /battcharger3S1/PH -> /battcharger4S/PH
- Q11 pad 1: /battcharger3S2/PH -> /battcharger3S1/PH
- Q11 pad 2: /battcharger3S2/PH -> /battcharger3S1/PH
- Q11 pad 3: /battcharger3S2/PH -> /battcharger3S1/PH
- Q11 pad 4: /battcharger3S2/HIDRV -> /battcharger3S1/HIDRV
- Q12 pad 4: /battcharger3S2/LODRV -> /battcharger3S1/LODRV
- Q12 pad 5: /battcharger3S2/PH -> /battcharger3S1/PH
- Q13 pad 1: /battcharger4S/PH -> /battcharger3S2/PH
- Q13 pad 2: /battcharger4S/PH -> /battcharger3S2/PH
- Q13 pad 3: /battcharger4S/PH -> /battcharger3S2/PH
- Q13 pad 4: /battcharger4S/HIDRV -> /battcharger3S2/HIDRV
- Q14 pad 4: /battcharger4S/LODRV -> /battcharger3S2/LODRV
- Q14 pad 5: /battcharger4S/PH -> /battcharger3S2/PH
- Q9 pad 1: /battcharger3S1/PH -> /battcharger4S/PH
- Q9 pad 2: /battcharger3S1/PH -> /battcharger4S/PH
- Q9 pad 3: /battcharger3S1/PH -> /battcharger4S/PH
- Q9 pad 4: /battcharger3S1/HIDRV -> /battcharger4S/HIDRV
- R17 pad 1: /battcharger3S1/Vref -> /battcharger4S/Vref
- R19 pad 2: /battcharger3S1/Vfb -> /battcharger4S/Vfb
- R20 pad 2: /battcharger3S1/Vfb -> /battcharger4S/Vfb
- R21 pad 1: /battcharger3S1/Vfb -> /battcharger4S/Vfb
- R22 pad 2: /battcharger3S1/ISET1 -> /battcharger4S/ISET1
- R23 pad 1: /battcharger3S1/ISET1 -> /battcharger4S/ISET1
- R24 pad 2: /battcharger3S1/ISET1 -> /battcharger4S/ISET1
- R25 pad 1: /battcharger3S1/ISET1 -> /battcharger4S/ISET1
- R26 pad 1: /battcharger3S1/CSRP -> /battcharger4S/CSRP
- R26 pad 2: /battcharger3S1/CSRN -> /battcharger4S/CSRN
- R27 pad 2: /battcharger3S1/ISET2 -> /battcharger4S/ISET2
- R28 pad 1: /battcharger3S1/ISET2 -> /battcharger4S/ISET2
- R29 pad 2: /battcharger3S1/ISET2 -> /battcharger4S/ISET2
- R30 pad 1: /battcharger3S1/ISET2 -> /battcharger4S/ISET2
- R36 pad 1: /battcharger3S2/Vref -> /battcharger3S1/Vref
- R38 pad 2: /battcharger3S2/Vfb -> /battcharger3S1/Vfb
- R39 pad 2: /battcharger3S2/Vfb -> /battcharger3S1/Vfb
- R40 pad 1: /battcharger3S2/Vfb -> /battcharger3S1/Vfb
- R41 pad 2: /battcharger3S2/ISET1 -> /battcharger3S1/ISET1
- R42 pad 1: /battcharger3S2/ISET1 -> /battcharger3S1/ISET1
- R43 pad 2: /battcharger3S2/ISET1 -> /battcharger3S1/ISET1
- R44 pad 1: /battcharger3S2/ISET1 -> /battcharger3S1/ISET1
- R45 pad 1: /battcharger3S2/CSRP -> /battcharger3S1/CSRP
- R45 pad 2: /battcharger3S2/CSRN -> /battcharger3S1/CSRN
- R46 pad 2: /battcharger3S2/ISET2 -> /battcharger3S1/ISET2
- R47 pad 1: /battcharger3S2/ISET2 -> /battcharger3S1/ISET2
- R48 pad 2: /battcharger3S2/ISET2 -> /battcharger3S1/ISET2
- R49 pad 1: /battcharger3S2/ISET2 -> /battcharger3S1/ISET2
- R55 pad 1: /battcharger4S/Vref -> /battcharger3S2/Vref
- R57 pad 2: /battcharger4S/Vfb -> /battcharger3S2/Vfb
- R58 pad 2: /battcharger4S/Vfb -> /battcharger3S2/Vfb
- R59 pad 1: /battcharger4S/Vfb -> /battcharger3S2/Vfb
- R60 pad 2: /battcharger4S/ISET1 -> /battcharger3S2/ISET1
- R61 pad 1: /battcharger4S/ISET1 -> /battcharger3S2/ISET1
- R62 pad 2: /battcharger4S/ISET1 -> /battcharger3S2/ISET1
- R63 pad 1: /battcharger4S/ISET1 -> /battcharger3S2/ISET1
- R64 pad 1: /battcharger4S/CSRP -> /battcharger3S2/CSRP
- R64 pad 2: /battcharger4S/CSRN -> /battcharger3S2/CSRN
- R65 pad 2: /battcharger4S/ISET2 -> /battcharger3S2/ISET2
- R66 pad 1: /battcharger4S/ISET2 -> /battcharger3S2/ISET2
- R67 pad 2: /battcharger4S/ISET2 -> /battcharger3S2/ISET2
- R68 pad 1: /battcharger4S/ISET2 -> /battcharger3S2/ISET2
- SW1 pad 2: /battcharger3S1/CSRN -> /battcharger4S/CSRN
- SW2 pad 2: /battcharger3S1/Vref -> /battcharger4S/Vref
- SW2 pad 5: /battcharger3S1/Vref -> /battcharger4S/Vref
- SW3 pad 2: /battcharger3S2/CSRN -> /battcharger3S1/CSRN
- SW4 pad 2: /battcharger3S2/Vref -> /battcharger3S1/Vref
- SW4 pad 5: /battcharger3S2/Vref -> /battcharger3S1/Vref
- SW5 pad 2: /battcharger4S/CSRN -> /battcharger3S2/CSRN
- SW6 pad 2: /battcharger4S/Vref -> /battcharger3S2/Vref
- SW6 pad 5: /battcharger4S/Vref -> /battcharger3S2/Vref
- U1 pad 10: /battcharger3S1/Vref -> /battcharger4S/Vref
- U1 pad 11: /battcharger3S1/ISET1 -> /battcharger4S/ISET1
- U1 pad 12: /battcharger3S1/Vfb -> /battcharger4S/Vfb
- U1 pad 13: /battcharger3S1/CSRN -> /battcharger4S/CSRN
- U1 pad 14: /battcharger3S1/CSRP -> /battcharger4S/CSRP
- U1 pad 15: /battcharger3S1/ISET2 -> /battcharger4S/ISET2
- U1 pad 16: /battcharger3S1/Vref -> /battcharger4S/Vref
- U1 pad 18: /battcharger3S1/REGN -> /battcharger4S/REGN
- U1 pad 19: /battcharger3S1/LODRV -> /battcharger4S/LODRV
- U1 pad 20: /battcharger3S1/PH -> /battcharger4S/PH
- U1 pad 21: /battcharger3S1/HIDRV -> /battcharger4S/HIDRV
- U1 pad 22: /battcharger3S1/BTST -> /battcharger4S/BTST
- U1 pad 4: /battcharger3S1/CE -> /CE1
- U1 pad 5: /CHG -> /CE
- U1 pad 8: /battcharger3S1/PG -> /battcharger4S/PG
- U1 pad 9: /battcharger3S1/STAT2 -> /battcharger4S/STAT2
- U2 pad 10: /battcharger3S2/Vref -> /battcharger3S1/Vref
- U2 pad 11: /battcharger3S2/ISET1 -> /battcharger3S1/ISET1
- U2 pad 12: /battcharger3S2/Vfb -> /battcharger3S1/Vfb
- U2 pad 13: /battcharger3S2/CSRN -> /battcharger3S1/CSRN
- U2 pad 14: /battcharger3S2/CSRP -> /battcharger3S1/CSRP
- U2 pad 15: /battcharger3S2/ISET2 -> /battcharger3S1/ISET2
- U2 pad 16: /battcharger3S2/Vref -> /battcharger3S1/Vref
- U2 pad 18: /battcharger3S2/REGN -> /battcharger3S1/REGN
- U2 pad 19: /battcharger3S2/LODRV -> /battcharger3S1/LODRV
- U2 pad 20: /battcharger3S2/PH -> /battcharger3S1/PH
- U2 pad 21: /battcharger3S2/HIDRV -> /battcharger3S1/HIDRV
- U2 pad 22: /battcharger3S2/BTST -> /battcharger3S1/BTST
- U2 pad 4: /battcharger3S2/CE -> /battcharger3S1/CE
- U2 pad 8: /battcharger3S2/PG -> /battcharger3S1/PG
- U2 pad 9: /battcharger3S2/STAT2 -> /battcharger3S1/STAT2
- U3 pad 10: /battcharger4S/Vref -> /battcharger3S2/Vref
- U3 pad 11: /battcharger4S/ISET1 -> /battcharger3S2/ISET1
- U3 pad 12: /battcharger4S/Vfb -> /battcharger3S2/Vfb
- U3 pad 13: /battcharger4S/CSRN -> /battcharger3S2/CSRN
- U3 pad 14: /battcharger4S/CSRP -> /battcharger3S2/CSRP
- U3 pad 15: /battcharger4S/ISET2 -> /battcharger3S2/ISET2
- U3 pad 16: /battcharger4S/Vref -> /battcharger3S2/Vref
- U3 pad 18: /battcharger4S/REGN -> /battcharger3S2/REGN
- U3 pad 19: /battcharger4S/LODRV -> /battcharger3S2/LODRV
- U3 pad 20: /battcharger4S/PH -> /battcharger3S2/PH
- U3 pad 21: /battcharger4S/HIDRV -> /battcharger3S2/HIDRV
- U3 pad 22: /battcharger4S/BTST -> /battcharger3S2/BTST
- U3 pad 4: /CE1 -> /battcharger3S2/CE
- U3 pad 5: /CE -> /CHG
- U3 pad 8: /battcharger4S/PG -> /battcharger3S2/PG
- U3 pad 9: /battcharger4S/STAT2 -> /battcharger3S2/STAT2
Routing:
- net VAA: track 40.0 -> 134.6 mm, vias 2 -> 3
- net GND: track 59.1 -> 33.0 mm, vias 6 -> 120
- net /battcharger4S/CSRN: track 0.00 -> 21.0 mm
- net /battcharger4S/PH: track 0.00 -> 18.4 mm, vias 0 -> 2
- net /battcharger4S/LODRV: track 0.00 -> 15.0 mm, vias 0 -> 2
- net /battcharger4S/HIDRV: track 0.00 -> 10.2 mm, vias 0 -> 2
- net /battcharger4S/BTST: track 0.00 -> 7.87 mm
- net Net-(C4-Pad1): track 0.00 -> 1.50 mm
- net +BATT: vias 0 -> 19
- added copper zone on F.Cu, net +BATT
- added copper zone on F.Cu, net /battcharger4S/CSRP
- added copper zone on F.Cu, net /battcharger4S/PH
- added copper zone on F.Cu, net VAA

Commit message: lab 28/10
Parts:
- removed R16, R35, R54: 100k, Resistor_SMD:R_0603_1608Metric
- R19, R38, R57: value 500k -> 700k
- R20, R39, R58: value 700k -> 500k
- R22, R41, R60: value 57.6k -> 76.8k
- R23, R42, R61: value 44.2k -> 26.1k
- R24, R43, R62: value 76.8k -> 57.6k
- R25, R44, R63: value 26.1k -> 44.2k
- moved D12 56.3 mm to (54.0, 70.4), turned to 180 degrees
- moved D13 56.2 mm to (54.0, 72.8), turned to 180 degrees
- moved D14 56.2 mm to (54.0, 75.2), turned to 180 degrees
- moved R13 46.9 mm to (51.0, 70.4), turned to 180 degrees
- moved R14 46.9 mm to (51.0, 72.8), turned to 180 degrees
- moved R15 46.9 mm to (51.0, 75.2), turned to 180 degrees
- moved SW1 38.3 mm to (70.9, 48.7)
- moved R20 33.3 mm to (70.9, 52.6), turned to -90 degrees
- moved R21 29.2 mm to (76.9, 52.6), turned to 90 degrees
- moved R19 28.6 mm to (74.9, 52.6), turned to -90 degrees
- moved C13 25.9 mm to (72.9, 52.6), turned to -90 degrees
- moved R23 24.0 mm to (112.6, 52.2), turned to 90 degrees
- moved SW2 21.5 mm to (107.3, 54.8)
- moved R22 21.1 mm to (111.0, 52.2), turned to -90 degrees
- moved C10 19.8 mm to (100.6, 55.0), turned to 90 degrees
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Connections:
- C10 pad 1: /battcharger4S/CSRN -> /battcharger4S/CSRP
- C25 pad 1: /battcharger3S1/CSRN -> /battcharger3S1/CSRP
- C40 pad 1: /battcharger3S2/CSRN -> /battcharger3S2/CSRP
Routing:
- net /battcharger4S/CSRN: track 21.0 -> 85.3 mm
- net /battcharger4S/CSRP: track 0.00 -> 58.3 mm
- net /CE1: track 32.3 -> 74.6 mm, vias 2 -> 4
- net /battcharger4S/Vref: track 0.00 -> 41.3 mm, vias 0 -> 2
- net /CE: track 0.00 -> 39.2 mm, vias 0 -> 2
- net /battcharger4S/Vfb: track 0.00 -> 34.7 mm, vias 0 -> 2
- net /battcharger4S/ISET1: track 0.00 -> 33.5 mm, vias 0 -> 2
- net /battcharger4S/ISET2: track 0.00 -> 28.8 mm, vias 0 -> 2
- net VAA: track 134.6 -> 158.0 mm, vias 3 -> 4
- net /battcharger4S/REGN: track 0.00 -> 8.53 mm
- net Net-(SW2A-A): track 0.00 -> 5.09 mm
- net Net-(SW2A-C): track 0.00 -> 5.09 mm
- net Net-(SW2B-C): track 0.00 -> 5.08 mm
- net Net-(SW2B-A): track 0.00 -> 5.08 mm
- net Net-(U1-TS): track 0.00 -> 3.61 mm
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Other:
- board text added: "ACTIVE CHARGING CHARGED"
- board text added: "SW2 Left: 7.2A Right: 4.2A"
- board text added: "SW7/SW1 Left: 4S Right: 3S"
- board text removed: "SW7 Left: 4S Right: 3S"
- board text removed: "SW8 Left: 4S Right: 3S"
- board text removed: "SW9 Left: 4S Right: 3S"

Commit message: local 28/10
Parts:
- added G***: LOGO, LOGO, F.Cu at (47.0, 73.2)
- added G***: LOGO, LOGO, F.Cu at (35.0, 138.0)
- added G***: LOGO, LOGO, F.Cu at (114.0, 113.2)
- added G***: LOGO, LOGO, F.Cu at (24.8, 35.0)
- added G***: LOGO, LOGO, F.Cu at (115.4, 34.3)
- D1, Q1, R1: moved to B.Cu
- Q27, Q28, Q29, Q30: footprint Package_SON:VSONP-8-1EP_5x6_P1.27mm -> Package_TO_SOT_SMD:TDSON-8-1
- Q5, Q6, Q7, Q8: footprint Package_TO_SOT_SMD:SOT-23-3 -> Package_TO_SOT_SMD:SOT-23
- moved C79 77.9 mm to (152.9, 125.5)
- moved C83 77.9 mm to (152.9, 135.5)
- moved C84 77.9 mm to (152.9, 138.0)
- moved C85 77.9 mm to (156.9, 125.5)
- moved C93 77.9 mm to (156.9, 135.5)
- moved C94 77.9 mm to (156.9, 138.0)
- moved D28 77.9 mm to (146.7, 132.6)
- moved R117 77.9 mm to (160.9, 125.5)
- moved R121 77.9 mm to (160.9, 135.5)
- moved R122 77.9 mm to (160.9, 138.0)
- moved R123 77.9 mm to (164.9, 125.5)
- moved R127 77.9 mm to (164.9, 135.5)
- moved U7 77.9 mm to (162.9, 146.6)
- moved C80 77.9 mm to (152.9, 128.0)
- moved C81 77.9 mm to (152.9, 130.5)
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Connections:
- Q15 pad 1: Net-(Q15-D) -> /battprot1/DSG
- Q15 pad 2: /battprot1/DSG -> GND
- Q15 pad 3: GND -> Net-(Q15-S)
- Q16 pad 4: Net-(Q15-D) -> Net-(Q15-S)
- Q17 pad 1: Net-(Q17-D) -> /CE1
- Q17 pad 2: /CE1 -> GND
- Q17 pad 3: GND -> Net-(Q17-S)
- Q18 pad 4: Net-(Q17-D) -> Net-(Q17-S)
- Q19 pad 1: Net-(Q19-D) -> /battprot2/DSG
- Q19 pad 2: /battprot2/DSG -> GND
- Q19 pad 3: GND -> Net-(Q19-S)
- Q20 pad 4: Net-(Q19-D) -> Net-(Q19-S)
- Q21 pad 1: Net-(Q21-D) -> /CE2
- Q21 pad 2: /CE2 -> GND
- Q21 pad 3: GND -> Net-(Q21-S)
- Q22 pad 4: Net-(Q21-D) -> Net-(Q21-S)
- Q23 pad 1: Net-(Q23-D) -> /battprot3/DSG
- Q23 pad 2: /battprot3/DSG -> GND
- Q23 pad 3: GND -> Net-(Q23-S)
- Q24 pad 4: Net-(Q23-D) -> Net-(Q23-S)
- Q25 pad 1: Net-(Q25-D) -> /CE3
- Q25 pad 2: /CE3 -> GND
- Q25 pad 3: GND -> Net-(Q25-S)
- Q26 pad 4: Net-(Q25-D) -> Net-(Q25-S)
- Q27 pad 1: +BATT -> /buckboost/SW1
- Q27 pad 2: /buckboost/HDRV1 -> /buckboost/SW1
- Q28 pad 1: /buckboost/SW1 -> /buckboost/CS
- Q28 pad 2: /buckboost/LDRV1 -> /buckboost/CS
- Q29 pad 1: /buckboost/Vout -> /buckboost/SW2
- Q29 pad 2: /buckboost/HDRV2 -> /buckboost/SW2
- Q30 pad 1: /buckboost/SW2 -> /buckboost/CS
- Q30 pad 2: /buckboost/LDRV2 -> /buckboost/CS
- Q5 pad 1: Net-(D8-A) -> Net-(J3-Pin_1)
- Q5 pad 2: Net-(J3-Pin_1) -> GND
- Q5 pad 3: GND -> Net-(D8-A)
- Q6 pad 1: Net-(D9-A) -> Net-(J3-Pin_2)
- Q6 pad 2: Net-(J3-Pin_2) -> GND
- Q6 pad 3: GND -> Net-(D9-A)
- Q7 pad 1: Net-(D10-A) -> Net-(J3-Pin_3)
- Q7 pad 2: Net-(J3-Pin_3) -> GND
- Q7 pad 3: GND -> Net-(D10-A)
- Q8 pad 1: Net-(D11-A) -> Net-(J3-Pin_4)
- Q8 pad 2: Net-(J3-Pin_4) -> GND
- Q8 pad 3: GND -> Net-(D11-A)
- R113 pad 2: Net-(Q23-D) -> Net-(Q23-S)
- R115 pad 2: Net-(Q25-D) -> Net-(Q25-S)
- R81 pad 2: Net-(Q15-D) -> Net-(Q15-S)
- R83 pad 2: Net-(Q17-D) -> Net-(Q17-S)
- R97 pad 2: Net-(Q19-D) -> Net-(Q19-S)
- R99 pad 2: Net-(Q21-D) -> Net-(Q21-S)
Routing:
- net VAA: track 158.0 -> 510.9 mm, vias 4 -> 9
- net /CHG: track 0.00 -> 352.2 mm, vias 0 -> 8
- net /CE2: track 30.2 -> 361.5 mm, vias 2 -> 5
- net /battcharger3S1/PG: track 0.00 -> 300.8 mm, vias 0 -> 4
- net /battcharger3S1/STAT2: track 0.00 -> 291.2 mm, vias 0 -> 4
- net /CE3: track 30.3 -> 225.5 mm, vias 2 -> 3
- net /battcharger3S2/PG: track 0.00 -> 149.4 mm, vias 0 -> 2
- net /battcharger3S2/STAT2: track 0.00 -> 146.1 mm, vias 0 -> 2
- net /battcharger3S2/CSRN: track 0.00 -> 120.9 mm
- net /battcharger3S1/CSRN: track 0.00 -> 101.9 mm
- net /CE: track 39.2 -> 138.8 mm, vias 2 -> 4
- net +BATT: track 0.00 -> 86.3 mm
- net /battcharger3S1/CSRP: track 0.00 -> 58.3 mm
- net /battcharger3S2/CSRP: track 0.00 -> 58.3 mm
- net /battcharger4S/PG: track 2.37 -> 54.9 mm
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- added copper zone on B.Cu, net +BATT
- added copper zone on F.Cu, net /battcharger3S1/CSRP
- added copper zone on F.Cu, net /battcharger3S1/PH
- added copper zone on F.Cu, net /battcharger3S2/CSRP
- added copper zone on F.Cu, net /battcharger3S2/PH
- added copper zone on B.Cu, net Net-(J1-Pin_1)
- removed copper zone on F.Cu, net Net-(J1-Pin_1)
Other:
- board text added: "BATT1 ACTIVE CHARGING CHARGED"
- board text added: "BATT2 ACTIVE CHARGING CHARGED"
- board text added: "BATT3 ACTIVE CHARGING CHARGED"
- board text added: "Long Live 2 8"
- board text added: "SW4 Left: 7.2A Right: 4.2A"
- board text added: "SW6 Left: 7.2A Right: 4.2A"
- board text added: "SW8/SW3 Left: 4S Right: 3S"
- board text added: "SW9/SW5 Left: 4S Right: 3S"
- board text added: "by Helushka"
- board text removed: "ACTIVE CHARGING CHARGED"
