File: powerdist/buck_v0.1.kicad_sch (KiCad schematic)
At the start: 7 parts, among them U9 TPS56637RPAR

Commit message: local 13/10
Parts:
- added R55: 10k, symbol Device:R_Small_US
- renumbered C88 to C51, C89 to C52, C86 to C53, C91 to C54, C93 to C55, R118 to R56, U9 to U5
Connections:
- net FB: now also R55.2
- net GND: now also R55.1

Commit message: local 14/10
Parts:
- U5: footprint RPA0010A -> powerdist:RPA0010A
Changed lines of the file:
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@@
 		(dnp no)
 		(fields_autoplaced yes)
-		(property "Reference" "#FLG022"
+		(property "Reference" "#FLG017"
 			(at 175.26 89.535 0)
 			(effects
@@
 			(project "powerdist"
 				(path "/d8b3361c-0c6a-4299-baf2-0b5966ddedfb/754cc4f7-7309-49ec-a85a-88e49e6da610/d20406a8-849c-4daf-91e9-f6a00db06dfe"
-					(reference "#FLG023")
-					(unit 1)
-				)
-				(path "/d8b3361c-0c6a-4299-baf2-0b5966ddedfb/754cc4f7-7309-49ec-a85a-88e49e6da610/e120752a-0fbf-4556-b9bd-c9acc7dc7af6"
-					(reference "#FLG022")
+					(reference "#FLG017")
+					(unit 1)
+				)
+				(path "/d8b3361c-0c6a-4299-baf2-0b5966ddedfb/754cc4f7-7309-49ec-a85a-88e49e6da610/e120752a-0fbf-4556-b9bd-c9acc7dc7af6"
+					(reference "#FLG014")
 					(unit 1)
 				)
@@
 			)
 		)
-		(property "Footprint" "RPA0010A"
+		(property "Footprint" "powerdist:RPA0010A"
 			(at 140.97 82.55 0)
 			(effects
@@
 		(dnp no)
 		(fields_autoplaced yes)
-		(property "Reference" "#FLG020"
+		(property "Reference" "#FLG016"
 			(at 162.56 81.915 0)
 			(effects
@@
 			(project "powerdist"
 				(path "/d8b3361c-0c6a-4299-baf2-0b5966ddedfb/754cc4f7-7309-49ec-a85a-88e49e6da610/d20406a8-849c-4daf-91e9-f6a00db06dfe"
-					(reference "#FLG021")
-					(unit 1)
-				)
-				(path "/d8b3361c-0c6a-4299-baf2-0b5966ddedfb/754cc4f7-7309-49ec-a85a-88e49e6da610/e120752a-0fbf-4556-b9bd-c9acc7dc7af6"
-					(reference "#FLG020")
+					(reference "#FLG016")
+					(unit 1)
+				)
+				(path "/d8b3361c-0c6a-4299-baf2-0b5966ddedfb/754cc4f7-7309-49ec-a85a-88e49e6da610/e120752a-0fbf-4556-b9bd-c9acc7dc7af6"
+					(reference "#FLG013")
 					(unit 1)
 				)
@@
 		(dnp no)
 		(fields_autoplaced yes)
-		(property "Reference" "#FLG018"
+		(property "Reference" "#FLG015"
 			(at 161.29 67.945 0)
 			(effects
@@
 			(project "powerdist"
 				(path "/d8b3361c-0c6a-4299-baf2-0b5966ddedfb/754cc4f7-7309-49ec-a85a-88e49e6da610/d20406a8-849c-4daf-91e9-f6a00db06dfe"
-					(reference "#FLG019")
-					(unit 1)
-				)
-				(path "/d8b3361c-0c6a-4299-baf2-0b5966ddedfb/754cc4f7-7309-49ec-a85a-88e49e6da610/e120752a-0fbf-4556-b9bd-c9acc7dc7af6"
-					(reference "#FLG018")
-					(unit 1)
-				)
+					(reference "#FLG015")
+					(unit 1)
+				)
+				(path "/d8b3361c-0c6a-4299-baf2-0b5966ddedfb/754cc4f7-7309-49ec-a85a-88e49e6da610/e120752a-0fbf-4556-b9bd-c9acc7dc7af6"
+					(reference "#FLG012")
+					(unit 1)
+				)

Commit message: local 19/10
Parts:
- renumbered C51 to C55, C52 to C56, C53 to C57, C54 to C58, C55 to C59
Changed lines of the file:
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@@
 		(dnp no)
 		(fields_autoplaced yes)
-		(property "Reference" "C54"
+		(property "Reference" "C58"
 			(at 163.83 72.3962 0)
 			(effects
@@
 			(project "powerdist"
 				(path "/d8b3361c-0c6a-4299-baf2-0b5966ddedfb/754cc4f7-7309-49ec-a85a-88e49e6da610/d20406a8-849c-4daf-91e9-f6a00db06dfe"
-					(reference "C54")
-					(unit 1)
-				)
-				(path "/d8b3361c-0c6a-4299-baf2-0b5966ddedfb/754cc4f7-7309-49ec-a85a-88e49e6da610/e120752a-0fbf-4556-b9bd-c9acc7dc7af6"
-					(reference "C49")
+					(reference "C58")
+					(unit 1)
+				)
+				(path "/d8b3361c-0c6a-4299-baf2-0b5966ddedfb/754cc4f7-7309-49ec-a85a-88e49e6da610/e120752a-0fbf-4556-b9bd-c9acc7dc7af6"
+					(reference "C53")
 					(unit 1)
 				)
@@
 		(dnp no)
 		(fields_autoplaced yes)
-		(property "Reference" "C51"
+		(property "Reference" "C55"
 			(at 99.06 71.9581 0)
 			(effects
@@
 			(project "powerdist"
 				(path "/d8b3361c-0c6a-4299-baf2-0b5966ddedfb/754cc4f7-7309-49ec-a85a-88e49e6da610/d20406a8-849c-4daf-91e9-f6a00db06dfe"
-					(reference "C51")
-					(unit 1)
-				)
-				(path "/d8b3361c-0c6a-4299-baf2-0b5966ddedfb/754cc4f7-7309-49ec-a85a-88e49e6da610/e120752a-0fbf-4556-b9bd-c9acc7dc7af6"
-					(reference "C46")
+					(reference "C55")
+					(unit 1)
+				)
+				(path "/d8b3361c-0c6a-4299-baf2-0b5966ddedfb/754cc4f7-7309-49ec-a85a-88e49e6da610/e120752a-0fbf-4556-b9bd-c9acc7dc7af6"
+					(reference "C50")
 					(unit 1)
 				)
@@
 		(dnp no)
 		(fields_autoplaced yes)
-		(property "Reference" "C53"
+		(property "Reference" "C57"
 			(at 116.84 72.3962 0)
 			(effects
@@
 			(project "powerdist"
 				(path "/d8b3361c-0c6a-4299-baf2-0b5966ddedfb/754cc4f7-7309-49ec-a85a-88e49e6da610/d20406a8-849c-4daf-91e9-f6a00db06dfe"
-					(reference "C53")
-					(unit 1)
-				)
-				(path "/d8b3361c-0c6a-4299-baf2-0b5966ddedfb/754cc4f7-7309-49ec-a85a-88e49e6da610/e120752a-0fbf-4556-b9bd-c9acc7dc7af6"
-					(reference "C48")
+					(reference "C57")
+					(unit 1)
+				)
+				(path "/d8b3361c-0c6a-4299-baf2-0b5966ddedfb/754cc4f7-7309-49ec-a85a-88e49e6da610/e120752a-0fbf-4556-b9bd-c9acc7dc7af6"
+					(reference "C52")
 					(unit 1)
 				)
@@
 		(dnp no)
 		(fields_autoplaced yes)
-		(property "Reference" "C55"
+		(property "Reference" "C59"
 			(at 171.45 82.5562 0)
 			(effects
@@
 			(project "powerdist"
 				(path "/d8b3361c-0c6a-4299-baf2-0b5966ddedfb/754cc4f7-7309-49ec-a85a-88e49e6da610/d20406a8-849c-4daf-91e9-f6a00db06dfe"
-					(reference "C55")
-					(unit 1)
-				)
-				(path "/d8b3361c-0c6a-4299-baf2-0b5966ddedfb/754cc4f7-7309-49ec-a85a-88e49e6da610/e120752a-0fbf-4556-b9bd-c9acc7dc7af6"
-					(reference "C50")
+					(reference "C59")
+					(unit 1)
+				)
+				(path "/d8b3361c-0c6a-4299-baf2-0b5966ddedfb/754cc4f7-7309-49ec-a85a-88e49e6da610/e120752a-0fbf-4556-b9bd-c9acc7dc7af6"
+					(reference "C54")
 					(unit 1)
 				)
@@
 		(dnp no)
 		(fields_autoplaced yes)
-		(property "Reference" "C52"
+		(property "Reference" "C56"
 			(at 107.95 71.9581 0)
 			(effects
@@
 			(project "powerdist"
 				(path "/d8b3361c-0c6a-4299-baf2-0b5966ddedfb/754cc4f7-7309-49ec-a85a-88e49e6da610/d20406a8-849c-4daf-91e9-f6a00db06dfe"
-					(reference "C52")
-					(unit 1)
-				)
-				(path "/d8b3361c-0c6a-4299-baf2-0b5966ddedfb/754cc4f7-7309-49ec-a85a-88e49e6da610/e120752a-0fbf-4556-b9bd-c9acc7dc7af6"
-					(reference "C47")
-					(unit 1)
-				)
+					(reference "C56")
+					(unit 1)
+				)
+				(path "/d8b3361c-0c6a-4299-baf2-0b5966ddedfb/754cc4f7-7309-49ec-a85a-88e49e6da610/e120752a-0fbf-4556-b9bd-c9acc7dc7af6"
+					(reference "C51")
+					(unit 1)
+				)

Commit message: lab 20/10
Parts:
- renumbered R55 to R58, R56 to R59
Changed lines of the file:
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@@
 		(dnp no)
 		(fields_autoplaced yes)
-		(property "Reference" "R55"
+		(property "Reference" "R58"
 			(at 166.37 90.1699 0)
 			(effects
@@
 			(project "powerdist"
 				(path "/d8b3361c-0c6a-4299-baf2-0b5966ddedfb/754cc4f7-7309-49ec-a85a-88e49e6da610/d20406a8-849c-4daf-91e9-f6a00db06dfe"
-					(reference "R55")
-					(unit 1)
-				)
-				(path "/d8b3361c-0c6a-4299-baf2-0b5966ddedfb/754cc4f7-7309-49ec-a85a-88e49e6da610/e120752a-0fbf-4556-b9bd-c9acc7dc7af6"
-					(reference "R53")
+					(reference "R58")
+					(unit 1)
+				)
+				(path "/d8b3361c-0c6a-4299-baf2-0b5966ddedfb/754cc4f7-7309-49ec-a85a-88e49e6da610/e120752a-0fbf-4556-b9bd-c9acc7dc7af6"
+					(reference "R56")
 					(unit 1)
 				)
@@
 		(dnp no)
 		(fields_autoplaced yes)
-		(property "Reference" "R56"
+		(property "Reference" "R59"
 			(at 172.72 73.66 90)
 			(effects
@@
 			(project "powerdist"
 				(path "/d8b3361c-0c6a-4299-baf2-0b5966ddedfb/754cc4f7-7309-49ec-a85a-88e49e6da610/d20406a8-849c-4daf-91e9-f6a00db06dfe"
-					(reference "R56")
-					(unit 1)
-				)
-				(path "/d8b3361c-0c6a-4299-baf2-0b5966ddedfb/754cc4f7-7309-49ec-a85a-88e49e6da610/e120752a-0fbf-4556-b9bd-c9acc7dc7af6"
-					(reference "R54")
-					(unit 1)
-				)
+					(reference "R59")
+					(unit 1)
+				)
+				(path "/d8b3361c-0c6a-4299-baf2-0b5966ddedfb/754cc4f7-7309-49ec-a85a-88e49e6da610/e120752a-0fbf-4556-b9bd-c9acc7dc7af6"
+					(reference "R57")
+					(unit 1)
+				)

Commit message: lab 21/10
Parts:
- R58, R59: footprint (none) -> Resistor_SMD:R_0603_1608Metric
Changed lines of the file:
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@@
 			)
 		)
-		(property "Footprint" ""
+		(property "Footprint" "Resistor_SMD:R_0603_1608Metric"
 			(at 163.83 91.44 0)
 			(effects
@@
 			)
 		)
-		(property "Footprint" ""
+		(property "Footprint" "Resistor_SMD:R_0603_1608Metric"
 			(at 172.72 80.01 0)
 			(effects

Commit message: lab 23/10
Parts:
- C55, C56: footprint (none) -> Capacitor_SMD:C_0603_1608Metric; symbol Device:C_Polarized_Small_US -> Device:C_Small
- C57, C58, C59: footprint (none) -> Capacitor_SMD:C_0603_1608Metric
Changed lines of the file:
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@@
 			)
 		)
-		(property "Footprint" ""
+		(property "Footprint" "Capacitor_SMD:C_0603_1608Metric"
 			(at 161.29 73.66 0)
 			(effects
@@
 	)
 	(symbol
-		(lib_id "Device:C_Polarized_Small_US")
+		(lib_id "Device:C_Small")
 		(at 96.52 73.66 0)
 		(unit 1)
@@
 		(fields_autoplaced yes)
 		(property "Reference" "C55"
-			(at 99.06 71.9581 0)
+			(at 99.06 72.3962 0)
 			(effects
 				(font
@@
 		)
 		(property "Value" "10u"
-			(at 99.06 74.4981 0)
+			(at 99.06 74.9362 0)
 			(effects
 				(font
@@
 			)
 		)
-		(property "Footprint" ""
+		(property "Footprint" "Capacitor_SMD:C_0603_1608Metric"
 			(at 96.52 73.66 0)
 			(effects
@@
 			)
 		)
-		(property "Description" "Polarized capacitor, small US symbol"
+		(property "Description" "Unpolarized capacitor, small symbol"
 			(at 96.52 73.66 0)
 			(effects
@@
 			)
 		)
-		(property "Footprint" ""
+		(property "Footprint" "Capacitor_SMD:C_0603_1608Metric"
 			(at 114.3 73.66 0)
 			(effects
@@
 			)
 		)
-		(property "Footprint" ""
+		(property "Footprint" "Capacitor_SMD:C_0603_1608Metric"
 			(at 168.91 83.82 0)
 			(effects
@@
 	)
 	(symbol
-		(lib_id "Device:C_Polarized_Small_US")
+		(lib_id "Device:C_Small")
 		(at 105.41 73.66 0)
 		(unit 1)
@@
 		(fields_autoplaced yes)
 		(property "Reference" "C56"
-			(at 107.95 71.9581 0)
+			(at 107.95 72.3962 0)
 			(effects
 				(font
@@
 		)
 		(property "Value" "10u"
-			(at 107.95 74.4981 0)
+			(at 107.95 74.9362 0)
 			(effects
 				(font
@@
 			)
 		)
-		(property "Footprint" ""
+		(property "Footprint" "Capacitor_SMD:C_0603_1608Metric"
 			(at 105.41 73.66 0)
 			(effects
@@
 			)
 		)
-		(property "Description" "Polarized capacitor, small US symbol"
+		(property "Description" "Unpolarized capacitor, small symbol"
 			(at 105.41 73.66 0)
 			(effects

Commit message: local 26/10
Parts:
- renumbered C55 to C103, C56 to C104, C57 to C105, C58 to C106, C59 to C107, R58 to R129, R59 to R130, U5 to U10
Connections:
- net +12V renamed Vin

Commit message: lab 30/10: DONE
Parts:
- U10: footprint powerdist:RPA0010A -> powerdist:CONV_TPS56637RPAR
Changed lines of the file:
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@@
 			)
 		)
-		(property "Footprint" "powerdist:RPA0010A"
+		(property "Footprint" "powerdist:CONV_TPS56637RPAR"
 			(at 140.97 82.55 0)
 			(effects
