File: powerdist/powerdist.kicad_sch (KiCad schematic)
At the start: 0 parts

Commit message: local 26/10
Parts:
- added BATT1, BATT2, BATT3: Conn_01x02_Socket, Connector:Banana_Jack_2Pin, symbol Connector:Conn_01x02_Socket
- added BATT3S1, BATT3S2, BATT3S3: Conn_01x03_Pin, Connector_JST:JST_XH_B4B-XH-AM_1x04_P2.50mm_Vertical, symbol Connector:Conn_01x04_Pin
- added BATT4S1, BATT4S2, BATT4S3: Conn_01x04_Pin, Connector_JST:JST_XH_B5B-XH-AM_1x05_P2.50mm_Vertical, symbol Connector:Conn_01x05_Pin
- added C1, C2, C3: 47u, Capacitor_SMD:C_1206_3216Metric, symbol Device:C_Small
- added D1, D2, D3, D4: BZT52, Diode_SMD:D_SOD-123, symbol Device:D_Zener_Small_Filled
- added D10, D11, D8, D9: 10BQ030, Diode_SMD:D_SMB, symbol Device:D_Schottky_Small_Filled
- added D5, D6, D7: 1N4148W, Diode_SMD:D_SOD-123, symbol Device:D_Small_Filled
- added F1, F2, F3, F4: 3544-2, powerdist:CONN_3544-2_KEY, symbol 3544-2:3544-2
- added J1, J2: Conn_01x02_Socket, TerminalBlock:TerminalBlock_bornier-2_P5.08mm, symbol Connector:Screw_Terminal_01x02
- added J10, J11, J12, J13: Conn_01x02_Pin, Connector_PinHeader_2.54mm:PinHeader_1x02_P2.54mm_Vertical, symbol Connector:Conn_01x02_Pin
- added J3, J9: Conn_01x04_Socket, Connector_JST:JST_XH_B4B-XH-AM_1x04_P2.50mm_Vertical, symbol Connector:Conn_01x04_Socket
- added J4: Conn_01x04_Pin, Connector_PinHeader_2.54mm:PinHeader_1x04_P2.54mm_Vertical, symbol Connector:Conn_01x04_Pin
- added J5, J6, J7, J8: Conn_01x02_Socket, Connector_JST:JST_XH_B2B-XH-AM_1x02_P2.50mm_Vertical, symbol Connector:Conn_01x02_Socket
- added L1: 5.6u, Inductor_SMD:L_Vishay_IHLP-5050, symbol Device:L_Small
- added L2: 3.3u, Inductor_SMD:L_Vishay_IHLP-5050, symbol Device:L_Small
- added Q1, Q2, Q3, Q4: SI4178DY, Package_SO:PowerPAK_SO-8_Single, symbol Transistor_FET:Si7336ADP
- added Q5, Q6, Q7, Q8: DMN2056U, Package_TO_SOT_SMD:SOT-23-3, symbol Simulation_SPICE:NMOS
- added R1, R10, R11, R2, R3, R4: 1k, Resistor_SMD:R_0603_1608Metric, symbol Device:R_Small_US
- added R5, R8, R9: 20k, Resistor_SMD:R_0603_1608Metric, symbol Device:R_Small_US
- added R6: 115k, Resistor_SMD:R_0603_1608Metric, symbol Device:R_Small_US
- added R7: 75k, Resistor_SMD:R_0603_1608Metric, symbol Device:R_Small_US
Connections:
- new net: D1.1 (K), Q1.4 (G), R1.2
- new net: J1.1 (Pin_1), Q1.5 (D)
- new net: D4.1 (K), Q4.4 (G), R4.2
- new net: BATT3.1 (Pin_1), Q4.5 (D)
- new net: D9.2 (A), J6.1 (Pin_1), Q6.1 (D)
- new net: F1.1, F1.2, J1.2 (Pin_2)
- new net: D2.1 (K), Q2.4 (G), R2.2
- new net: D10.2 (A), J7.1 (Pin_1), Q7.1 (D)
- new net: D11.2 (A), J8.1 (Pin_1), Q8.1 (D)
- new net: J3.2 (Pin_2), Q6.2 (G)
- new net: D8.2 (A), J5.1 (Pin_1), Q5.1 (D)
- new net: J3.1 (Pin_1), Q5.2 (G)
- new net: D3.1 (K), Q3.4 (G), R3.2
- new net: J3.4 (Pin_4), Q8.2 (G)
- new net: BATT1.1 (Pin_1), Q2.5 (D)
- new net: BATT2.1 (Pin_1), Q3.5 (D)
- new net: BATT2.2 (Pin_2), F3.1, F3.2
- new net: J3.3 (Pin_3), Q7.2 (G)
- new net: BATT3.2 (Pin_2), F4.1, F4.2
- new net: BATT1.2 (Pin_2), F2.1, F2.2
- new net +12V: D10.1 (K), D11.1 (K), D8.1 (K), D9.1 (K), J5.2 (Pin_2), J6.2 (Pin_2), J7.2 (Pin_2), J8.2 (Pin_2)
- new net +3V3: J4.1 (Pin_1), J9.1 (Pin_1), R10.1, R11.1
- new net +5V: C2.1, J2.1 (Pin_1), L2.1, R7.1
- new net +7.5V: C1.1, C3.1, L1.1, R6.1
- new net +BATT: R5.1
- new net 1BATT-: BATT3S1.4 (Pin_4), BATT4S1.5 (Pin_5)
- new net 1BATT1: BATT3S1.3 (Pin_3), BATT4S1.4 (Pin_4)
- new net 1BATT2: BATT3S1.2 (Pin_2), BATT4S1.3 (Pin_3)
- new net 1BATT3: BATT3S1.1 (Pin_1), BATT4S1.2 (Pin_2)
- new net 1BATT4: BATT4S1.1 (Pin_1)
- new net 2BATT-: BATT3S2.4 (Pin_4), BATT4S2.5 (Pin_5)
- new net 2BATT1: BATT3S2.3 (Pin_3), BATT4S2.4 (Pin_4)
- new net 2BATT2: BATT3S2.2 (Pin_2), BATT4S2.3 (Pin_3)
- new net 2BATT3: BATT3S2.1 (Pin_1), BATT4S2.2 (Pin_2)
- new net 2BATT4: BATT4S2.1 (Pin_1)
- new net 3BATT-: BATT3S3.4 (Pin_4), BATT4S3.5 (Pin_5)
- new net 3BATT1: BATT3S3.3 (Pin_3), BATT4S3.4 (Pin_4)
- new net 3BATT2: BATT3S3.2 (Pin_2), BATT4S3.3 (Pin_3)
- new net 3BATT3: BATT3S3.1 (Pin_1), BATT4S3.2 (Pin_2)
- new net 3BATT4: BATT4S3.1 (Pin_1)
- new net CE: D5.1 (K), D6.1 (K), D7.1 (K)
- new net CE2: R8.1
- new net CE3: R9.1
- new net CHG: D7.2 (A), R5.2
- new net GND: C1.2, C2.2, C3.2, D1.2 (A), J10.2 (Pin_2), J11.2 (Pin_2), J12.2 (Pin_2), J13.2 (Pin_2), J2.2 (Pin_2), J4.4 (Pin_4), J9.4 (Pin_4), Q1.1 (S), Q1.2 (S), Q1.3 (S), Q5.3 (S), Q6.3 (S), Q7.3 (S), Q8.3 (S)
- new net S1: J10.1 (Pin_1)
- new net S2: J11.1 (Pin_1)
- new net S3: J12.1 (Pin_1)
- new net S4: J13.1 (Pin_1)
- new net SCL: J4.3 (Pin_3), J9.3 (Pin_3), R11.2
- new net SDA: J4.2 (Pin_2), J9.2 (Pin_2), R10.2
- new net VAA: F1.3, F1.4, R1.1
- new net Vbatt1: F2.3, F2.4, R2.1
- new net Vbatt1-: D2.2 (A), Q2.1 (S), Q2.2 (S), Q2.3 (S)
- new net Vbatt2: F3.3, F3.4, R3.1
- new net Vbatt2-: D3.2 (A), Q3.1 (S), Q3.2 (S), Q3.3 (S)
- new net Vbatt3: F4.3, F4.4, R4.1
- new net Vbatt3-: D4.2 (A), Q4.1 (S), Q4.2 (S), Q4.3 (S)
- new net battcharger3S1/CE: D5.2 (A), R8.2
- new net battcharger3S2/CE: D6.2 (A), R9.2
- new net buck5V1/FB: R7.2
- new net buck5V1/Vout: L2.2
- new net buck7V5/FB: R6.2
- new net buck7V5/Vout: L1.2
- no-connect marks 0 -> 3
Other:
- removed sheet v0.1
- added sheet ADCpower (adc_v0.1.kicad_sch)
- added sheet ADCstall (adc_v0.1.kicad_sch)
- added sheet battcharger3S1 (battcharge_v0.2.kicad_sch)
- added sheet battcharger3S2 (battcharge_v0.2.kicad_sch)
- added sheet battcharger4S (battcharge_v0.2.kicad_sch)
- added sheet battprot1 (battprot_v0.2.kicad_sch)
- added sheet battprot2 (battprot_v0.2.kicad_sch)
- added sheet battprot3 (battprot_v0.2.kicad_sch)
- added sheet buck5V1 (buck_v0.1.kicad_sch)
- added sheet buck7V5 (buck_v0.1.kicad_sch)
- added sheet buckboost (buckboost_v0.1.kicad_sch)
- added sheet power monitor (monitor_v0.1.kicad_sch)
- added sheet stall monitor1 (monitor_v0.1.kicad_sch)
- added sheet stall monitor2 (monitor_v0.1.kicad_sch)
- added sheet stall monitor3 (monitor_v0.1.kicad_sch)
- added sheet stall monitor4 (monitor_v0.1.kicad_sch)
- note added: "FROM RPI"
- note added: "TO MOTORS"
- note added: "TO RPI"
- note added: "TO SERVO CONTROL"
- title: MASTER SHEET -> powerdist

Commit message: lab 27/10
Other:
- moved on the sheet: R5

Commit message: local 28/10
Parts:
- Q5, Q6, Q7, Q8: footprint Package_TO_SOT_SMD:SOT-23-3 -> Package_TO_SOT_SMD:SOT-23; symbol Simulation_SPICE:NMOS -> Transistor_FET:DMN2056U
Connections:
- net GND: now also Q5.2 (S), Q6.2 (S), Q7.2 (S), Q8.2 (S); no longer Q5.3 (S), Q6.3 (S), Q7.3 (S), Q8.3 (S)
- net at D9.2 (A), J6.1 (Pin_1): now also Q6.3 (D); no longer Q6.1 (D)
- net at D10.2 (A), J7.1 (Pin_1): now also Q7.3 (D); no longer Q7.1 (D)
- net at D11.2 (A), J8.1 (Pin_1): now also Q8.3 (D); no longer Q8.1 (D)
- net at J3.2 (Pin_2): now also Q6.1 (G); no longer Q6.2 (G)
- net at D8.2 (A), J5.1 (Pin_1): now also Q5.3 (D); no longer Q5.1 (D)
- net at J3.1 (Pin_1): now also Q5.1 (G); no longer Q5.2 (G)
- net at J3.4 (Pin_4): now also Q8.1 (G); no longer Q8.2 (G)
- net at J3.3 (Pin_3): now also Q7.1 (G); no longer Q7.2 (G)
Changed lines of the file:
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@@
 	)
 	(symbol
-		(lib_id "Simulation_SPICE:NMOS")
+		(lib_id "Transistor_FET:DMN2056U")
 		(at 374.65 133.35 0)
 		(unit 1)
@@
 			)
 		)
-		(property "Footprint" "Package_TO_SOT_SMD:SOT-23-3"
-			(at 379.73 130.81 0)
+		(property "Footprint" "Package_TO_SOT_SMD:SOT-23"
+			(at 379.73 135.255 0)
 			(effects
 				(font
 					(size 1.27 1.27)
+					(italic yes)
 				)
+				(justify left)
 				(hide yes)
 			)
 		)
-		(property "Datasheet" "https://ngspice.sourceforge.io/docs/ngspice-html-manual/manual.xhtml#cha_MOSFETs"
-			(at 374.65 146.05 0)
+		(property "Datasheet" "http://www.diodes.com/assets/Datasheets/DMN2056U.pdf"
+			(at 379.73 137.16 0)
 			(effects
 				(font
 					(size 1.27 1.27)
 				)
+				(justify left)
 				(hide yes)
 			)
 		)
-		(property "Description" "N-MOSFET transistor, drain/source/gate"
+		(property "Description" "4A Id, 20V Vds, N-Channel MOSFET, SOT-23"
 			(at 374.65 133.35 0)
 			(effects
@@
 	)
 	(symbol
-		(lib_id "Simulation_SPICE:NMOS")
+		(lib_id "Transistor_FET:DMN2056U")
 		(at 374.65 106.68 0)
 		(unit 1)
@@
 			)
 		)
-		(property "Footprint" "Package_TO_SOT_SMD:SOT-23-3"
-			(at 379.73 104.14 0)
+		(property "Footprint" "Package_TO_SOT_SMD:SOT-23"
+			(at 379.73 108.585 0)
 			(effects
 				(font
 					(size 1.27 1.27)
+					(italic yes)
 				)
+				(justify left)
 				(hide yes)
 			)
 		)
-		(property "Datasheet" "https://ngspice.sourceforge.io/docs/ngspice-html-manual/manual.xhtml#cha_MOSFETs"
-			(at 374.65 119.38 0)
+		(property "Datasheet" "http://www.diodes.com/assets/Datasheets/DMN2056U.pdf"
+			(at 379.73 110.49 0)
 			(effects
 				(font
 					(size 1.27 1.27)
 				)
+				(justify left)
 				(hide yes)
 			)
 		)
-		(property "Description" "N-MOSFET transistor, drain/source/gate"
+		(property "Description" "4A Id, 20V Vds, N-Channel MOSFET, SOT-23"
 			(at 374.65 106.68 0)
 			(effects
@@
 	)
 	(symbol
-		(lib_id "Simulation_SPICE:NMOS")
+		(lib_id "Transistor_FET:DMN2056U")
 		(at 374.65 186.69 0)
 		(unit 1)
@@
 			)
 		)
-		(property "Footprint" "Package_TO_SOT_SMD:SOT-23-3"
-			(at 379.73 184.15 0)
+		(property "Footprint" "Package_TO_SOT_SMD:SOT-23"
+			(at 379.73 188.595 0)
 			(effects
 				(font
 					(size 1.27 1.27)
+					(italic yes)
 				)
+				(justify left)
 				(hide yes)
 			)
 		)
-		(property "Datasheet" "https://ngspice.sourceforge.io/docs/ngspice-html-manual/manual.xhtml#cha_MOSFETs"
-			(at 374.65 199.39 0)
+		(property "Datasheet" "http://www.diodes.com/assets/Datasheets/DMN2056U.pdf"
+			(at 379.73 190.5 0)
 			(effects
 				(font
 					(size 1.27 1.27)
 				)
+				(justify left)
 				(hide yes)
 			)
 		)
-		(property "Description" "N-MOSFET transistor, drain/source/gate"
+		(property "Description" "4A Id, 20V Vds, N-Channel MOSFET, SOT-23"
 			(at 374.65 186.69 0)
 			(effects
@@
 	)
 	(symbol
-		(lib_id "Simulation_SPICE:NMOS")
+		(lib_id "Transistor_FET:DMN2056U")
 		(at 374.65 160.02 0)
 		(unit 1)
@@
 			)
 		)
-		(property "Footprint" "Package_TO_SOT_SMD:SOT-23-3"
-			(at 379.73 157.48 0)
+		(property "Footprint" "Package_TO_SOT_SMD:SOT-23"
+			(at 379.73 161.925 0)
 			(effects
 				(font
 					(size 1.27 1.27)
+					(italic yes)
 				)
+				(justify left)
 				(hide yes)
 			)
 		)
-		(property "Datasheet" "https://ngspice.sourceforge.io/docs/ngspice-html-manual/manual.xhtml#cha_MOSFETs"
-			(at 374.65 172.72 0)
+		(property "Datasheet" "http://www.diodes.com/assets/Datasheets/DMN2056U.pdf"
+			(at 379.73 163.83 0)
 			(effects
 				(font
 					(size 1.27 1.27)
 				)
+				(justify left)
 				(hide yes)
 			)
 		)
-		(property "Description" "N-MOSFET transistor, drain/source/gate"
+		(property "Description" "4A Id, 20V Vds, N-Channel MOSFET, SOT-23"
 			(at 374.65 160.02 0)
 			(effects

Commit message: local 29/10
Parts:
- added J14: Conn_01x04_Pin, Connector_PinHeader_2.54mm:PinHeader_1x04_P2.54mm_Vertical, symbol Connector:Conn_01x04_Pin
- D10, D11, D8, D9: value 10BQ030 -> XBS053V13R; footprint Diode_SMD:D_SMB -> Diode_SMD:D_SOD-323_HandSoldering
- J10, J11, J12, J13: value Conn_01x02_Pin -> Conn_01x03_Pin; footprint Connector_PinHeader_2.54mm:PinHeader_1x02_P2.54mm_Vertical -> Connector_PinHeader_2.54mm:PinHeader_1x03_P2.54mm_Vertical; symbol Connector:Conn_01x02_Pin -> Connector:Conn_01x03_Pin
Connections:
- net GND: now also J10.3 (Pin_3), J11.3 (Pin_3), J12.3 (Pin_3), J13.3 (Pin_3); no longer J10.2 (Pin_2), J11.2 (Pin_2), J12.2 (Pin_2), J13.2 (Pin_2)
- net S1: now also J10.2 (Pin_2); no longer J10.1 (Pin_1)
- net S2: now also J11.2 (Pin_2); no longer J11.1 (Pin_1)
- net S3: now also J12.2 (Pin_2); no longer J12.1 (Pin_1)
- net S4: now also J13.2 (Pin_2); no longer J13.1 (Pin_1)
- new net: J10.1 (Pin_1), J14.1 (Pin_1)
- new net: J13.1 (Pin_1), J14.4 (Pin_4)
- new net: J12.1 (Pin_1), J14.3 (Pin_3)
- new net: J11.1 (Pin_1), J14.2 (Pin_2)
Other:
- note added: "FROM SERVO CONTROL"
- note added: "TO SERVOS"
- moved on the sheet: J2, J3

Commit message: lab 30/10: DONE
Parts:
- J3: footprint Connector_JST:JST_XH_B4B-XH-AM_1x04_P2.50mm_Vertical -> Connector_PinHeader_2.54mm:PinHeader_1x04_P2.54mm_Vertical
- J9: value Conn_01x04_Socket -> Conn_01x04_Pin; footprint Connector_JST:JST_XH_B4B-XH-AM_1x04_P2.50mm_Vertical -> Connector_PinHeader_2.54mm:PinHeader_1x04_P2.54mm_Vertical; symbol Connector:Conn_01x04_Socket -> Connector:Conn_01x04_Pin
Changed lines of the file:
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@@
 	)
 	(symbol
-		(lib_id "Connector:Conn_01x04_Socket")
+		(lib_id "Connector:Conn_01x04_Pin")
 		(at 389.89 27.94 0)
+		(mirror y)
 		(unit 1)
 		(exclude_from_sim no)
@@
 		(dnp no)
 		(property "Reference" "J9"
-			(at 385.318 34.798 0)
+			(at 387.096 34.544 0)
 			(effects
 				(font
@@
 			)
 		)
-		(property "Value" "Conn_01x04_Socket"
-			(at 385.318 37.338 0)
+		(property "Value" "Conn_01x04_Pin"
+			(at 392.43 36.83 0)
 			(effects
 				(font
 					(size 1.27 1.27)
 				)
-				(justify left)
 			)
 		)
-		(property "Footprint" "Connector_JST:JST_XH_B4B-XH-AM_1x04_P2.50mm_Vertical"
+		(property "Footprint" "Connector_PinHeader_2.54mm:PinHeader_1x04_P2.54mm_Vertical"
 			(at 389.89 27.94 0)
 			(effects
@@
 		)
 		(instances
-			(project ""
+			(project "powerdist"
 				(path "/d8b3361c-0c6a-4299-baf2-0b5966ddedfb"
 					(reference "J9")
@@
 			)
 		)
-		(property "Footprint" "Connector_JST:JST_XH_B4B-XH-AM_1x04_P2.50mm_Vertical"
+		(property "Footprint" "Connector_PinHeader_2.54mm:PinHeader_1x04_P2.54mm_Vertical"
 			(at 351.79 144.78 0)
 			(effects
@@
 			)
 		)
-		(pin "SENSE1" input
+		(pin "SENSE4" input
 			(at 224.79 213.36 180)
 			(effects
@@
 			)
 		)
-		(pin "SENSE2" input
+		(pin "SENSE3" input
 			(at 224.79 215.9 180)
 			(effects
@@
 			)
 		)
-		(pin "SENSE3" input
+		(pin "SENSE1" input
 			(at 266.7 213.36 0)
 			(effects
@@
 			)
 		)
-		(pin "SENSE4" input
+		(pin "SENSE2" input
 			(at 266.7 215.9 0)
 			(effects

Commit message: local 30/10
Parts:
- added J15: Conn_01x02_Socket, TerminalBlock:TerminalBlock_bornier-2_P5.08mm, symbol Connector:Conn_01x02_Socket
- added Q31: DMN2056U, Package_TO_SOT_SMD:SOT-23, symbol Transistor_FET:DMN2056U
- added R16: 20k, Resistor_SMD:R_0603_1608Metric, symbol Device:R_Small_US
Connections:
- net +BATT: now also R16.1
- net CHG: now also Q31.3 (D)
- net GND: now also J15.1 (Pin_1), Q31.2 (S)
- new net: J15.2 (Pin_2), Q31.1 (G), R16.2
Other:
- note added: "TO ESTOP"

Commit message: lab 27/11
Other:
- note added: "INCORPORATE - LF - SONAR - MOTOR REVERSE - LED"
Changed lines of the file:
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@@
+		)
+	)
+	(text "INCORPORATE\n- LF\n- SONAR\n- MOTOR REVERSE\n- LED"
+		(exclude_from_sim no)
+		(at 381.254 262.128 0)
+		(effects
+			(font
+				(size 1.27 1.27)
+			)
+			(justify left)
 		)
 	)

Commit message: lab 29/11
Other:
- note added: "INCORPORATE - LF - SONAR - MOTOR REVERSE - LED BATTPROT ISSUES BUCKBOOST ISSUES"
- note removed: "INCORPORATE - LF - SONAR - MOTOR REVERSE - LED"
Changed lines of the file:
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@@
 		)
 	)
-	(text "INCORPORATE\n- LF\n- SONAR\n- MOTOR REVERSE\n- LED"
+	(text "INCORPORATE\n- LF\n- SONAR\n- MOTOR REVERSE\n- LED\nBATTPROT ISSUES\nBUCKBOOST ISSUES"
 		(exclude_from_sim no)
-		(at 381.254 262.128 0)
+		(at 381.254 261.112 0)
 		(effects
 			(font
