File: powerdist/powerdist.kicad_sch (KiCad schematic)
At the start: 65 parts, among them J1 Conn_01x02_Socket, J10 Conn_01x03_Pin, J11 Conn_01x03_Pin, J12 Conn_01x03_Pin, J13 Conn_01x03_Pin, J14 Conn_01x04_Pin, J15 Conn_01x02_Socket, J2 Conn_01x02_Socket, J3 Conn_01x04_Socket, J4 Conn_01x04_Pin, J5 Conn_01x02_Socket, J6 Conn_01x02_Socket, J7 Conn_01x02_Socket, J8 Conn_01x02_Socket, J9 Conn_01x04_Pin, Q1 SI4178DY, Q2 SI4178DY, Q3 SI4178DY, Q31 DMN2056U, Q4 SI4178DY, Q5 DMN2056U, Q6 DMN2056U, Q7 DMN2056U, Q8 DMN2056U

Commit message: lab 06/12
Other:
- note added: "INCORPORATE - LF - MOTOR REVERSE - LED BATTPROT ISSUES BUCKBOOST ISSUES"
- note added: "Q31 SIGNAL FET BATTCHARGE ISSUES 3/4 LAYER PCB"
- note removed: "INCORPORATE - LF - SONAR - MOTOR REVERSE - LED BATTPROT ISSUES BUCKBOOST ISSUES"
Changed lines of the file:
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@@
 		)
 	)
-	(text "INCORPORATE\n- LF\n- SONAR\n- MOTOR REVERSE\n- LED\nBATTPROT ISSUES\nBUCKBOOST ISSUES"
+	(text "INCORPORATE\n- LF\n- MOTOR REVERSE\n- LED\nBATTPROT ISSUES\nBUCKBOOST ISSUES"
 		(exclude_from_sim no)
-		(at 381.254 261.112 0)
+		(at 361.696 261.112 0)
 		(effects
 			(font
+				(size 1.27 1.27)
+			)
+			(justify left)
+		)
+	)
+	(text "Q31 SIGNAL FET\nBATTCHARGE ISSUES\n3/4 LAYER PCB"
+		(exclude_from_sim no)
+		(at 382.778 258.572 0)
+		(effects
+			(font
