File: top/top.kicad_sch (KiCad schematic)
At the start: 1 part

Commit message: lab 06/12
Connections:
- net LF 5V: now also MCU1.4 (5V)
- net LF GND: now also MCU1.14 (GND)
- net LED DATA: now reaches MCU1.16 (GPIO23/SDIO_CMD)
- net M DIR: now reaches MCU1.31 (GPCLK2/GPIO06)
- no-connect marks 28 -> 24
Changed lines of the file:
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@@
-	)
-	(no_connect
-		(at 69.85 71.12)
-	)
-	(no_connect
-		(at 99.06 87.63)
 	)
 	(no_connect
@@
 	)
 	(no_connect
-		(at 135.89 36.83)
-	)
-	(no_connect
 		(at 69.85 78.74)
 	)
@@
 	)
 	(no_connect
-		(at 135.89 67.31)
-	)
-	(no_connect
 		(at 69.85 68.58)
 	)
@@
 		)
 	)
+	(global_label "LF 5V"
+		(shape input)
+		(at 135.89 36.83 0)
+		(fields_autoplaced yes)
+		(effects
+			(font
+				(size 1.27 1.27)
+			)
+			(justify left)
+		)
+		(property "Intersheetrefs" "${INTERSHEET_REFS}"
+			(at 144.2576 36.83 0)
+			(effects
+				(font
+					(size 1.27 1.27)
+				)
+				(justify left)
+				(hide yes)
+			)
+		)
+	)
+	(global_label "LED DATA"
+		(shape input)
+		(at 69.85 71.12 180)
+		(fields_autoplaced yes)
+		(effects
+			(font
+				(size 1.27 1.27)
+			)
+			(justify right)
+		)
+		(property "Intersheetrefs" "${INTERSHEET_REFS}"
+			(at 58.0353 71.12 0)
+			(effects
+				(font
+					(size 1.27 1.27)
+				)
+				(justify right)
+				(hide yes)
+			)
+		)
+	)
 	(global_label "M BR"
 		(shape input)
@@
 			(effects
 				(font
+					(size 1.27 1.27)
+				)
+				(justify left)
+				(hide yes)
+			)
+		)
+	)
+	(global_label "LF GND"
+		(shape input)
+		(at 99.06 87.63 270)
+		(fields_autoplaced yes)
+		(effects
+			(font
+				(size 1.27 1.27)
+			)
+			(justify right)
+		)
+		(property "Intersheetrefs" "${INTERSHEET_REFS}"
+			(at 99.06 97.57 90)
+			(effects
+				(font
+					(size 1.27 1.27)
+				)
+				(justify right)
+				(hide yes)
+			)
+		)
+	)
+	(global_label "M DIR"
+		(shape input)
+		(at 135.89 67.31 0)
+		(fields_autoplaced yes)
+		(effects
+			(font
+				(size 1.27 1.27)
+			)
+			(justify left)
+		)
+		(property "Intersheetrefs" "${INTERSHEET_REFS}"
+			(at 144.439 67.31 0)
+			(effects
+				(font

Commit message: lab 08/12
Connections:
- net M BR is gone; now on net M FR: MCU1.35 (GPIO19/SPI1_MISO/PCM_FS)
- net M FR: no longer MCU1.33 (GPIO13/PWM1)
- no-connect marks 24 -> 25
Other:
- note added: "DEAD PIN"
